File: mykeeb/pcb/mykeeb.kicad_pcb (KiCad board)
At the start: 2 copper layers, 159.5 x 119.1 mm, 130 parts, among them K0 KEYSW, K1 KEYSW, K10 KEYSW, K11 KEYSW, K12 KEYSW, K13 KEYSW, K14 KEYSW, K15 KEYSW, K16 KEYSW, K17 KEYSW, K2 KEYSW, K20 KEYSW, K21 KEYSW, K22 KEYSW, K23 KEYSW, K24 KEYSW, K25 KEYSW, K26 KEYSW, K27 KEYSW, K3 KEYSW, K30 KEYSW, K31 KEYSW, K32 KEYSW, K33 KEYSW, K34 KEYSW, K35 KEYSW, K36 KEYSW, K37 KEYSW, K4 KEYSW, K40 KEYSW, K44 KEYSW, K45 KEYSW, K46 KEYSW, K47 KEYSW, K5 KEYSW, K6 KEYSW, K7 KEYSW, SW1 SW_Push, U1 ProMicro

Commit message: order rev1
Signed-off-by: Maximilian Huber <gh@maxhbr.de>
Parts:
- added BT2: Conn_01x02, Connector_PinHeader_2.54mm:PinHeader_1x02_P2.54mm_Vertical, F.Cu at (173.0, 82.3)
- moved D15 1.19 mm to (151.2, 69.1)
- moved D25 1.19 mm to (151.2, 88.1)
- moved D35 1.19 mm to (151.2, 107.2)
- moved D36 1.19 mm to (172.6, 100.0)
- moved D45 1.19 mm to (136.9, 126.2)
- moved D5 1.19 mm to (151.2, 50.0)
- moved D0 1.19 mm to (56.0, 59.5)
- moved D10 1.19 mm to (56.0, 78.6)
- moved D12 1.19 mm to (94.1, 64.3)
- moved D13 1.19 mm to (113.1, 59.5)
- moved D2 1.19 mm to (94.1, 45.2)
- moved D21 1.19 mm to (75.0, 95.2)
- moved D22 1.19 mm to (94.1, 83.3)
- moved D23 1.19 mm to (113.1, 78.6)
- moved D3 1.19 mm to (113.1, 40.5)
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Routing:
- net GND: track 192.4 -> 8.20 mm, vias 2 -> 77
- net Net-(BT1-Pad1): track 47.4 -> 87.1 mm, vias 2 -> 3
- net row2: track 227.8 -> 193.1 mm, vias 3 -> 1
- net row0: track 345.1 -> 377.9 mm, vias 6 -> 3
- net col6: track 199.0 -> 217.1 mm, vias 2 -> 1
- net row3: track 208.0 -> 194.1 mm, vias 3 -> 1
- net row4: track 229.2 -> 215.4 mm, vias 2 -> 1
- net col3: track 220.9 -> 232.3 mm
- net Net-(D45-Pad1): track 51.1 -> 39.8 mm
- net Net-(D26-Pad1): track 38.2 -> 27.8 mm
- net Net-(D6-Pad1): track 38.2 -> 27.9 mm
- net Net-(D16-Pad1): track 38.2 -> 27.9 mm
- net Net-(D46-Pad1): track 71.0 -> 63.3 mm
- net col0: track 273.3 -> 280.8 mm
- net col1: track 254.3 -> 261.4 mm
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- added copper zone on B.Cu, net GND
- added copper zone on F.Cu, net GND
