File: mykeeb/pcb/mykeeb.kicad_sch (KiCad schematic)
At the start: 83 parts, among them K1 KEYSW, K10 KEYSW, K11 KEYSW, K12 KEYSW, K13 KEYSW, K14 KEYSW, K15 KEYSW, K16 KEYSW, K2 KEYSW, K20 KEYSW, K21 KEYSW, K22 KEYSW, K23 KEYSW, K24 KEYSW, K25 KEYSW, K26 KEYSW, K3 KEYSW, K30 KEYSW, K31 KEYSW, K32 KEYSW, K33 KEYSW, K34 KEYSW, K35 KEYSW, K36 KEYSW, K4 KEYSW, K40 KEYSW, K41 KEYSW, K42 KEYSW, K43 KEYSW, K44 KEYSW, K45 KEYSW, K46 KEYSW, K5 KEYSW, K6 KEYSW

Commit message: wip on mykeeb
Signed-off-by: Maximilian Huber <gh@maxhbr.de>
Parts:
- added BT1, BT2: (no value), symbol Device:Battery_Cell
- added K40b1, K43b1: KEYSW, keyswitches:Kailh_socket_MX_optional_reversible, symbol keyboard_parts:KEYSW
- added U2: ProMicro, Keebio-Parts:ArduinoProMicro-BackSide, symbol keebio:ProMicro
- D0, D1, D10, D11, D12, D13, D14, D15, D16, D2, D20, D21, D22, D23, D24, D25, D26, D3, D30, D31, D32, D33, D34, D35, D36, D4, D40, D41, D42, D43, D44, D45, D46, D5, D6: value (none) -> DIODE; footprint (none) -> Keebio-Parts:D_SOD123F
- FID1: value (none) -> Fiducial; footprint (none) -> Fiducial:Fiducial_1mm_Mask2mm
- H1: value (none) -> MountingHole; footprint (none) -> MountingHole:MountingHole_3.2mm_M3
- H5, H6, H7, H8: footprint MountingHole:MountingHole_3.2mm_M3 -> MountingHole:MountingHole_2.2mm_M2
- K0: value (none) -> KEYSW; footprint (none) -> keyswitches:Kailh_socket_MX_optional_reversible
- SW1: value (none) -> SW_Push; footprint (none) -> Keebio-Parts:SW_Tactile_SPST_Angled_MJTP1117
- U1: value (none) -> ProMicro; footprint (none) -> Keebio-Parts:ArduinoProMicro-BackSide
Connections:
- net Bat+: now also BT1.1 (+), BT2.1 (+), U2.24 (RAW)
- net RST: now also U2.22 (RST)
- net col0: now also K40b1.1, U2.19 (A2/PF5)
- net col1: now also U2.18 (A1/PF6)
- net col2: now also U2.17 (A0/PF7)
- net col3: now also K43b1.1, U2.16 (15/PB1)
- net col4: now also U2.15 (14/PB3)
- net col5: now also U2.14 (16/PB2)
- net col6: now also U2.13 (10/PB6)
- net row0: now also U2.8 (5/PC6)
- net row1: now also U2.9 (6/PD7)
- net row2: now also U2.10 (7/PE6)
- net row3: now also U2.11 (8/PB4)
- net row4: now also U2.12 (9/PB5)
- net at D43.1 (K), K43.2: now also K43b1.2
- net at D40.1 (K), K40.2: now also K40b1.2
- net +5V renamed GND
- net GND: now also BT1.2 (-), BT2.2 (-), U2.23 (GND), U2.3 (GND), U2.4 (GND)
- no-connect marks 7 -> 14
Other:
- moved on the sheet: FID1, FID2, FID3, H1, H2, H3, H4, H5, H6, H7, H8, SW1

Commit message: wip on mykeeb
Signed-off-by: Maximilian Huber <gh@maxhbr.de>
Parts:
- removed BT2: (no value), symbol Device:Battery_Cell
- BT1: value (none) -> Battery_Cell; footprint (none) -> Connector_JST:JST_PH_S2B-PH-K_1x02_P2.00mm_Horizontal
Changed lines of the file:
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@@
   (junction (at 168.91 111.76) (diameter 0) (color 0 0 0 0)
   )
-  (junction (at 237.49 132.08) (diameter 0) (color 0 0 0 0)
-  )
   (junction (at 54.61 60.96) (diameter 0) (color 0 0 0 0)
   )
@@
   )
   (junction (at 125.73 76.2) (diameter 0) (color 0 0 0 0)
-  )
-  (junction (at 237.49 119.38) (diameter 0) (color 0 0 0 0)
   )
   (junction (at 148.59 76.2) (diameter 0) (color 0 0 0 0)
@@
     (stroke (width 0) (type default) (color 0 0 0 0))
   )
-  (wire (pts (xy 237.49 132.08) (xy 256.54 132.08))
-    (stroke (width 0) (type default) (color 0 0 0 0))
-  )
   (wire (pts (xy 223.52 132.08) (xy 237.49 132.08))
     (stroke (width 0) (type default) (color 0 0 0 0))
@@
     (stroke (width 0) (type default) (color 0 0 0 0))
   )
-  (wire (pts (xy 256.54 119.38) (xy 256.54 121.92))
-    (stroke (width 0) (type default) (color 0 0 0 0))
-  )
   (wire (pts (xy 148.59 101.6) (xy 148.59 99.06))
     (stroke (width 0) (type default) (color 0 0 0 0))
@@
     (stroke (width 0) (type default) (color 0 0 0 0))
   )
-  (wire (pts (xy 256.54 132.08) (xy 256.54 129.54))
-    (stroke (width 0) (type default) (color 0 0 0 0))
-  )
   (wire (pts (xy 80.01 86.36) (xy 80.01 88.9))
     (stroke (width 0) (type default) (color 0 0 0 0))
@@
   )
   (wire (pts (xy 36.83 138.43) (xy 34.29 138.43))
-    (stroke (width 0) (type default) (color 0 0 0 0))
-  )
-  (wire (pts (xy 237.49 119.38) (xy 256.54 119.38))
     (stroke (width 0) (type default) (color 0 0 0 0))
   )
@@
   (symbol (lib_id "power:GND") (at 262.89 67.31 0) (unit 1)
     (in_bom yes) (on_board yes) (fields_autoplaced)
-    (property "Reference" "#PWR?" (id 0) (at 262.89 73.66 0)
+    (property "Reference" "#PWR0105" (id 0) (at 262.89 73.66 0)
       (effects (font (size 1.27 1.27)) hide)
     )
@@
       (effects (font (size 1.27 1.27)) (justify left))
     )
-    (property "Value" "" (id 1) (at 241.3 126.2379 0)
-      (effects (font (size 1.27 1.27)) (justify left))
-    )
-    (property "Footprint" "" (id 2) (at 237.49 125.476 90)
+    (property "Value" "Battery_Cell" (id 1) (at 241.3 126.2379 0)
+      (effects (font (size 1.27 1.27)) (justify left))
+    )
+    (property "Footprint" "Connector_JST:JST_PH_S2B-PH-K_1x02_P2.00mm_Horizontal" (id 2) (at 237.49 125.476 90)
       (effects (font (size 1.27 1.27)) hide)
     )
@@
   (symbol (lib_id "power:GND") (at 218.44 29.21 0) (unit 1)
     (in_bom yes) (on_board yes) (fields_autoplaced)
-    (property "Reference" "#PWR?" (id 0) (at 218.44 35.56 0)
-      (effects (font (size 1.27 1.27)) hide)
-    )
-    (property "Value" "" (id 1) (at 218.44 34.29 0))
+    (property "Reference" "#PWR0103" (id 0) (at 218.44 35.56 0)
+      (effects (font (size 1.27 1.27)) hide)
+    )
+    (property "Value" "GND" (id 1) (at 218.44 34.29 0))
     (property "Footprint" "" (id 2) (at 218.44 29.21 0)
       (effects (font (size 1.27 1.27)) hide)
@@
   (symbol (lib_id "power:GND") (at 218.44 69.85 0) (unit 1)
     (in_bom yes) (on_board yes) (fields_autoplaced)
-    (property "Reference" "#PWR?" (id 0) (at 218.44 76.2 0)
+    (property "Reference" "#PWR0102" (id 0) (at 218.44 76.2 0)
       (effects (font (size 1.27 1.27)) hide)
     )
@@
   (symbol (lib_id "power:GND") (at 220.98 72.39 0) (unit 1)
     (in_bom yes) (on_board yes) (fields_autoplaced)
-    (property "Reference" "#PWR?" (id 0) (at 220.98 78.74 0)
+    (property "Reference" "#PWR0101" (id 0) (at 220.98 78.74 0)
       (effects (font (size 1.27 1.27)) hide)
     )
@@
     (pin "2")
   )
-  (symbol (lib_id "Device:Battery_Cell") (at 256.54 127 0) (unit 1)
-    (in_bom yes) (on_board yes) (fields_autoplaced)
-    (property "Reference" "BT2" (id 0) (at 260.35 123.6979 0)
-      (effects (font (size 1.27 1.27)) (justify left))
-    )
-    (property "Value" "" (id 1) (at 260.35 126.2379 0)
-      (effects (font (size 1.27 1.27)) (justify left))
-    )
-    (property "Footprint" "" (id 2) (at 256.54 125.476 90)
-      (effects (font (size 1.27 1.27)) hide)
-    )
-    (property "Datasheet" "~" (id 3) (at 256.54 125.476 90)
-      (effects (font (size 1.27 1.27)) hide)
-    )
-    (pin "1")
-    (pin "2")
-  )
   (symbol (lib_id "power:GND") (at 242.57 110.49 0) (unit 1)
     (in_bom yes) (on_board yes) (fields_autoplaced)
-    (property "Reference" "#PWR?" (id 0) (at 242.57 116.84 0)
+    (property "Reference" "#PWR0106" (id 0) (at 242.57 116.84 0)
       (effects (font (size 1.27 1.27)) hide)
     )
@@
   (symbol (lib_id "power:GND") (at 223.52 132.08 0) (unit 1)
     (in_bom yes) (on_board yes) (fields_autoplaced)
-    (property "Reference" "#PWR?" (id 0) (at 223.52 138.43 0)
+    (property "Reference" "#PWR0107" (id 0) (at 223.52 138.43 0)
       (effects (font (size 1.27 1.27)) hide)
     )
@@
   (symbol (lib_id "power:GND") (at 262.89 26.67 0) (unit 1)
     (in_bom yes) (on_board yes) (fields_autoplaced)
-    (property "Reference" "#PWR?" (id 0) (at 262.89 33.02 0)
+    (property "Reference" "#PWR0108" (id 0) (at 262.89 33.02 0)
       (effects (font (size 1.27 1.27)) hide)
     )
@@
   (symbol (lib_id "power:GND") (at 220.98 31.75 0) (unit 1)
     (in_bom yes) (on_board yes) (fields_autoplaced)
-    (property "Reference" "#PWR?" (id 0) (at 220.98 38.1 0)
+    (property "Reference" "#PWR0104" (id 0) (at 220.98 38.1 0)
       (effects (font (size 1.27 1.27)) hide)
     )
@@
   )
   (symbol_instances
+    (path "/63af35e2-3d89-438a-88bc-62570cafdc1b"
+      (reference "#PWR0101") (unit 1) (value "GND") (footprint "")
+    )
+    (path "/60d6b424-95f8-4e29-9c98-624d483fd85d"
+      (reference "#PWR0102") (unit 1) (value "GND") (footprint "")
+    )
+    (path "/56e18408-09a1-4a82-8f35-b63924873641"
+      (reference "#PWR0103") (unit 1) (value "GND") (footprint "")
+    )
+    (path "/fa7871ab-904f-493b-9b04-1d3f9a9f74b3"
+      (reference "#PWR0104") (unit 1) (value "GND") (footprint "")
+    )
     (path "/34620792-17f3-4021-88e3-6b8f6560aedc"
-      (reference "#PWR?") (unit 1) (value "GND") (footprint "")
-    )
-    (path "/56e18408-09a1-4a82-8f35-b63924873641"
-      (reference "#PWR?") (unit 1) (value "GND") (footprint "")
-    )
-    (path "/60d6b424-95f8-4e29-9c98-624d483fd85d"
-      (reference "#PWR?") (unit 1) (value "GND") (footprint "")
-    )
-    (path "/63af35e2-3d89-438a-88bc-62570cafdc1b"
-      (reference "#PWR?") (unit 1) (value "GND") (footprint "")
+      (reference "#PWR0105") (unit 1) (value "GND") (footprint "")
     )
     (path "/d96d2f82-dc2a-44d4-a289-0118ed77d142"
-      (reference "#PWR?") (unit 1) (value "GND") (footprint "")
+      (reference "#PWR0106") (unit 1) (value "GND") (footprint "")
     )
     (path "/e07b29ed-0bd2-4e47-ae5f-d63f0c6c3fdc"
-      (reference "#PWR?") (unit 1) (value "GND") (footprint "")
+      (reference "#PWR0107") (unit 1) (value "GND") (footprint "")
     )
     (path "/e31b91a5-5c56-4320-8d33-f6fbe1327eb4"
-      (reference "#PWR?") (unit 1) (value "GND") (footprint "")
-    )
-    (path "/fa7871ab-904f-493b-9b04-1d3f9a9f74b3"
-      (reference "#PWR?") (unit 1) (value "GND") (footprint "")
+      (reference "#PWR0108") (unit 1) (value "GND") (footprint "")
     )
     (path "/442f53f2-39ff-41c2-a967-02f3186c8b37"
       (reference "BT1") (unit 1) (value "Battery_Cell") (footprint "Connector_JST:JST_PH_S2B-PH-K_1x02_P2.00mm_Horizontal")
     )
-    (path "/d8668d1f-712c-48ca-a843-abc3154cb335"
-      (reference "BT2") (unit 1) (value "Battery_Cell") (footprint "Connector_JST:JST_PH_S2B-PH-K_1x02_P2.00mm_Horizontal")
-    )
     (path "/e41759dc-e8b4-4683-8ab7-83c4b7632e4d"

Commit message: add v0.1 pcb
Signed-off-by: Maximilian Huber <gh@maxhbr.de>
Parts:
- removed U2: ProMicro, Keebio-Parts:ArduinoProMicro-BackSide, symbol keebio:ProMicro
- added D17, D27, D37, D47, D7: DIODE, Keebio-Parts:D_SOD123F, symbol pspice:DIODE
- added H10, H9: MountingHole, MountingHole:MountingHole_2.2mm_M2, symbol Mechanical:MountingHole
- added JPbat+a0, JPbat+b0, JPc0a1, JPc0b1, JPc1a1, JPc1b1, JPc2a1, JPc2b1, JPc3a1, JPc3b1, JPc4a1, JPc4b1, JPc5a1, JPc5b1, JPc6a1, JPc6b1, JPc7a1, JPc7b1, JPgbda0, JPgndb0, JPr0a1, JPr0b1, JPr1a1, JPr1b1, JPr2a1, JPr2b1, JPr3a1, JPr3b1, JPr4a1, JPr4b1, JPresa0, JPresb0: SolderJumper_2_Open, Jumper:SolderJumper-2_P1.3mm_Open_TrianglePad1.0x1.5mm, symbol Jumper:SolderJumper_2_Open
- added K17, K27, K37, K47: KEYSW, Button_Switch_THT:SW_PUSH_6mm_H8mm, symbol keyboard_parts:KEYSW
- added SWbat1, SWbat2: SW_SPST, Button_Switch_SMD:SW_SPDT_PCM12, symbol Switch:SW_SPDT
- H8: value MountingHole -> (none); footprint MountingHole:MountingHole_2.2mm_M2 -> (none)
- K0, K1, K10, K11, K12, K13, K14, K15, K2, K20, K21, K22, K23, K24, K25, K3, K30, K31, K32, K33, K34, K35, K36, K4, K40, K41, K42, K43, K43b1, K44, K5: footprint keyswitches:Kailh_socket_MX_optional_reversible -> mykeeb:Kailh_socket_MX_optional_reversible_1u
- K16, K26, K45, K46, K6: value KEYSW -> (none); footprint keyswitches:Kailh_socket_MX_optional_reversible -> (none)
- K7: renamed from K40b1; footprint keyswitches:Kailh_socket_MX_optional_reversible -> mykeeb:Kailh_socket_MX_optional_reversible_1u
- SW1: footprint Keebio-Parts:SW_Tactile_SPST_Angled_MJTP1117 -> Button_Switch_THT:SW_PUSH_6mm
Connections:
- net Bat+: now also JPbat+a0.2 (B), JPbat+b0.2 (B), SWbat1.2 (B), SWbat2.2 (B); no longer BT1.1 (+), U1.24 (RAW)
- net GND: now also JPgbda0.2 (B), JPgndb0.2 (B); no longer U1.23 (GND), U1.3 (GND), U1.4 (GND)
- net RST: now also JPresa0.2 (B), JPresb0.2 (B); no longer U1.22 (RST)
- net col0: now also JPc0a1.2 (B), JPc0b1.2 (B); no longer K7.1, U1.19 (A2/PF5)
- net col1: now also JPc1a1.2 (B), JPc1b1.2 (B); no longer U1.18 (A1/PF6)
- net col2: now also JPc2a1.2 (B), JPc2b1.2 (B); no longer U1.17 (A0/PF7)
- net col3: now also JPc3a1.2 (B), JPc3b1.2 (B); no longer U1.16 (15/PB1)
- net col4: now also JPc4a1.2 (B), JPc4b1.2 (B); no longer U1.15 (14/PB3)
- net col5: now also JPc5a1.2 (B), JPc5b1.2 (B); no longer U1.14 (16/PB2)
- net col6: now also JPc6a1.2 (B), JPc6b1.2 (B); no longer U1.13 (10/PB6)
- net row0: now also D7.2 (A), JPr0a1.2 (B), JPr0b1.2 (B); no longer U1.8 (5/PC6)
- net row1: now also D17.2 (A), JPr1a1.2 (B), JPr1b1.2 (B); no longer U1.9 (6/PD7)
- net row2: now also D27.2 (A), JPr2a1.2 (B), JPr2b1.2 (B); no longer U1.10 (7/PE6)
- net row3: now also D37.2 (A), JPr3a1.2 (B), JPr3b1.2 (B); no longer U1.11 (8/PB4)
- net row4: now also D47.2 (A), JPr4a1.2 (B), JPr4b1.2 (B); no longer U1.12 (9/PB5)
- net at U1.1 (TX0/PD3): now also JPbat+b0.1 (A)
- net at U1.2 (RX1/PD2): now also JPgndb0.1 (A)
- net c0b: now reaches U1.6 (3/PD0)
- net c0b: now also JPc0b1.1 (A)
- net c1b: now reaches U1.7 (4/PD4)
- net c1b: now also JPc1b1.1 (A), JPc7a1.1 (A)
- net at D40.1 (K), K40.2: no longer K7.2
- new net: D27.1 (K), K27.2
- new net: D47.1 (K), K47.2
- new net: D37.1 (K), K37.2
- new net: JPresa0.1 (A), U1.22 (RST)
- new net: JPgbda0.1 (A), U1.23 (GND)
- new net: JPbat+a0.1 (A), U1.24 (RAW)
- new net: JPresb0.1 (A), U1.3 (GND)
- new net: BT1.1 (+), SWbat1.1 (A), SWbat2.3 (C)
- new net: D7.1 (K), K7.2
- new net: D17.1 (K), K17.2
- new net c0a: JPc0a1.1 (A), U1.19 (A2/PF5)
- new net c1a: JPc1a1.1 (A), JPc7b1.1 (A), U1.18 (A1/PF6)
- new net c2a: JPc2a1.1 (A), JPr0b1.1 (A), U1.17 (A0/PF7)
- new net c2b: JPc2b1.1 (A), JPr0a1.1 (A), U1.8 (5/PC6)
- new net c3a: JPc3a1.1 (A), JPr1b1.1 (A), U1.16 (15/PB1)
- new net c3b: JPc3b1.1 (A), JPr1a1.1 (A), U1.9 (6/PD7)
- new net c4a: JPc4a1.1 (A), JPr2b1.1 (A), U1.15 (14/PB3)
- new net c4b: JPc4b1.1 (A), JPr2a1.1 (A), U1.10 (7/PE6)
- new net c5a: JPc5a1.1 (A), JPr3b1.1 (A), U1.14 (16/PB2)
- new net c5b: JPc5b1.1 (A), JPr3a1.1 (A), U1.11 (8/PB4)
- new net c6a: JPc6a1.1 (A), JPr4b1.1 (A), U1.13 (10/PB6)
- new net c6b: JPc6b1.1 (A), JPr4a1.1 (A), U1.12 (9/PB5)
- new net col7: JPc7a1.2 (B), JPc7b1.2 (B), K17.1, K27.1, K37.1, K47.1, K7.1
- no-connect marks 14 -> 6
Other:
- moved on the sheet: BT1, D0, D1, D10, D11, D12, D13, D14, D15, D16, D2, D20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

Commit message: WIP
Signed-off-by: Maximilian Huber <gh@maxhbr.de>
Parts:
- removed K43b1: KEYSW, mykeeb:Kailh_socket_MX_optional_reversible_1u, symbol keyboard_parts:KEYSW
- H5: value MountingHole -> (none); footprint MountingHole:MountingHole_2.2mm_M2 -> (none)
Other:
- moved on the sheet: FID1, FID2, FID3, H1, H10, H2, H3, H4, H5, H6, H7, H8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

Commit message: order rev1
Signed-off-by: Maximilian Huber <gh@maxhbr.de>
Parts:
- added BT2: (no value), symbol Connector_Generic:Conn_01x02
- H5, H8: value (none) -> MountingHole; footprint (none) -> MountingHole:MountingHole_3.2mm_M3
- K16, K45, K6: value (none) -> KEYSW; footprint (none) -> mykeeb:Kailh_socket_MX_optional_reversible_1.25u
- K26, K46: value (none) -> KEYSW; footprint (none) -> mykeeb:Kailh_socket_MX_optional_reversible_1.5u
Connections:
- net GND: now also BT2.1 (Pin_1)
- net at BT1.1 (+), SWbat1.1 (A), SWbat2.3 (C): now also BT2.2 (Pin_2)
Changed lines of the file:
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@@
   (junction (at 245.11 170.18) (diameter 0) (color 0 0 0 0)
   )
+  (junction (at 269.24 45.72) (diameter 0) (color 0 0 0 0)
+  )
   (junction (at 107.95 59.69) (diameter 0) (color 0 0 0 0)
   )
@@
     (stroke (width 0) (type default) (color 0 0 0 0))
   )
+  (wire (pts (xy 309.88 44.45) (xy 309.88 49.53))
+    (stroke (width 0) (type default) (color 0 0 0 0))
+  )
   (wire (pts (xy 361.95 220.98) (xy 361.95 223.52))
     (stroke (width 0) (type default) (color 0 0 0 0))
@@
     (stroke (width 0) (type default) (color 0 0 0 0))
   )
+  (wire (pts (xy 309.88 44.45) (xy 287.02 44.45))
+    (stroke (width 0) (type default) (color 0 0 0 0))
+  )
+  (wire (pts (xy 285.75 45.72) (xy 285.75 53.34))
+    (stroke (width 0) (type default) (color 0 0 0 0))
+  )
   (wire (pts (xy 270.51 185.42) (xy 270.51 182.88))
     (stroke (width 0) (type default) (color 0 0 0 0))
@@
     (stroke (width 0) (type default) (color 0 0 0 0))
   )
+  (wire (pts (xy 287.02 44.45) (xy 287.02 50.8))
+    (stroke (width 0) (type default) (color 0 0 0 0))
+  )
   (wire (pts (xy 290.83 195.58) (xy 290.83 220.98))
     (stroke (width 0) (type default) (color 0 0 0 0))
@@
     (stroke (width 0) (type default) (color 0 0 0 0))
   )
+  (wire (pts (xy 287.02 50.8) (xy 288.29 50.8))
+    (stroke (width 0) (type default) (color 0 0 0 0))
+  )
   (wire (pts (xy 379.73 119.38) (xy 382.27 119.38))
     (stroke (width 0) (type default) (color 0 0 0 0))
@@
     (stroke (width 0) (type default) (color 0 0 0 0))
   )
+  (wire (pts (xy 288.29 53.34) (xy 285.75 53.34))
+    (stroke (width 0) (type default) (color 0 0 0 0))
+  )
   (wire (pts (xy 250.19 220.98) (xy 247.65 220.98))
     (stroke (width 0) (type default) (color 0 0 0 0))
@@
     (stroke (width 0) (type default) (color 0 0 0 0))
   )
+  (wire (pts (xy 269.24 45.72) (xy 285.75 45.72))
+    (stroke (width 0) (type default) (color 0 0 0 0))
+  )
   (wire (pts (xy 227.33 195.58) (xy 224.79 195.58))
     (stroke (width 0) (type default) (color 0 0 0 0))
@@
       (effects (font (size 1.27 1.27)) (justify left))
     )
-    (property "Value" "" (id 1) (at 327.66 48.2599 0)
+    (property "Value" "MountingHole" (id 1) (at 327.66 48.2599 0)
       (effects (font (size 1.27 1.27)) (justify left))
     )
-    (property "Footprint" "" (id 2) (at 325.12 46.99 0)
+    (property "Footprint" "MountingHole:MountingHole_3.2mm_M3" (id 2) (at 325.12 46.99 0)
       (effects (font (size 1.27 1.27)) hide)
     )
@@
       (effects (font (size 1.27 1.27)) (justify left))
     )
-    (property "Value" "" (id 1) (at 327.66 53.3399 0)
+    (property "Value" "MountingHole" (id 1) (at 327.66 53.3399 0)
       (effects (font (size 1.27 1.27)) (justify left))
     )
-    (property "Footprint" "" (id 2) (at 325.12 52.07 0)
+    (property "Footprint" "MountingHole:MountingHole_3.2mm_M3" (id 2) (at 325.12 52.07 0)
       (effects (font (size 1.27 1.27)) hide)
     )
@@
       (effects (font (size 1.524 1.524)))
     )
-    (property "Value" "" (id 1) (at 349.25 147.32 0)
+    (property "Value" "KEYSW" (id 1) (at 349.25 147.32 0)
       (effects (font (size 1.524 1.524)) hide)
     )
-    (property "Footprint" "" (id 2) (at 349.25 144.78 0)
+    (property "Footprint" "mykeeb:Kailh_socket_MX_optional_reversible_1.25u" (id 2) (at 349.25 144.78 0)
       (effects (font (size 1.524 1.524)) hide)
     )
@@
       (effects (font (size 1.524 1.524)))
     )
-    (property "Value" "" (id 1) (at 326.39 223.52 0)
+    (property "Value" "KEYSW" (id 1) (at 326.39 223.52 0)
       (effects (font (size 1.524 1.524)) hide)
     )
-    (property "Footprint" "" (id 2) (at 326.39 220.98 0)
+    (property "Footprint" "mykeeb:Kailh_socket_MX_optional_reversible_1.25u" (id 2) (at 326.39 220.98 0)
       (effects (font (size 1.524 1.524)) hide)
     )
@@
       (effects (font (size 1.524 1.524)))
     )
-    (property "Value" "" (id 1) (at 349.25 121.92 0)
+    (property "Value" "KEYSW" (id 1) (at 349.25 121.92 0)
       (effects (font (size 1.524 1.524)) hide)
     )
-    (property "Footprint" "" (id 2) (at 349.25 119.38 0)
+    (property "Footprint" "mykeeb:Kailh_socket_MX_optional_reversible_1.25u" (id 2) (at 349.25 119.38 0)
       (effects (font (size 1.524 1.524)) hide)
     )
@@
     (pin "2")
   )
+  (symbol (lib_id "power:GND") (at 309.88 49.53 0) (unit 1)
+    (in_bom yes) (on_board yes) (fields_autoplaced)
+    (property "Reference" "#PWR0101" (id 0) (at 309.88 55.88 0)
+      (effects (font (size 1.27 1.27)) hide)
+    )
+    (property "Value" "GND" (id 1) (at 309.88 54.61 0))
+    (property "Footprint" "" (id 2) (at 309.88 49.53 0)
+      (effects (font (size 1.27 1.27)) hide)
+    )
+    (property "Datasheet" "" (id 3) (at 309.88 49.53 0)
+      (effects (font (size 1.27 1.27)) hide)
+    )
+    (pin "1")
+  )
   (symbol (lib_id "Jumper:SolderJumper_2_Open") (at 121.92 185.42 0) (unit 1)
     (in_bom yes) (on_board yes) (fields_autoplaced)
@@
       (effects (font (size 1.524 1.524)))
     )
-    (property "Value" "" (id 1) (at 349.25 172.72 0)
+    (property "Value" "KEYSW" (id 1) (at 349.25 172.72 0)
       (effects (font (size 1.524 1.524)) hide)
     )
-    (property "Footprint" "" (id 2) (at 349.25 170.18 0)
+    (property "Footprint" "mykeeb:Kailh_socket_MX_optional_reversible_1.5u" (id 2) (at 349.25 170.18 0)
       (effects (font (size 1.524 1.524)) hide)
     )
@@
       (effects (font (size 1.524 1.524)))
     )
-    (property "Value" "" (id 1) (at 349.25 223.52 0)
+    (property "Value" "KEYSW" (id 1) (at 349.25 223.52 0)
       (effects (font (size 1.524 1.524)) hide)
     )
-    (property "Footprint" "" (id 2) (at 349.25 220.98 0)
+    (property "Footprint" "mykeeb:Kailh_socket_MX_optional_reversible_1.5u" (id 2) (at 349.25 220.98 0)
       (effects (font (size 1.524 1.524)) hide)
     )
@@
     (pin "2")
   )
+  (symbol (lib_id "Connector_Generic:Conn_01x02") (at 293.37 50.8 0) (unit 1)
+    (in_bom yes) (on_board yes) (fields_autoplaced)
+    (property "Reference" "BT2" (id 0) (at 295.91 50.7999 0)
+      (effects (font (size 1.27 1.27)) (justify left))
+    )
+    (property "Value" "" (id 1) (at 295.91 53.3399 0)
+      (effects (font (size 1.27 1.27)) (justify left))
+    )
+    (property "Footprint" "" (id 2) (at 293.37 50.8 0)
+      (effects (font (size 1.27 1.27)) hide)
+    )
+    (property "Datasheet" "~" (id 3) (at 293.37 50.8 0)
+      (effects (font (size 1.27 1.27)) hide)
+    )
+    (pin "1")
+    (pin "2")
+  )
   (symbol (lib_id "pspice:DIODE") (at 224.79 203.2 270) (unit 1)
     (in_bom yes) (on_board yes) (fields_autoplaced)
@@
   )
   (symbol_instances
+    (path "/b78adea6-6003-4b94-acc8-e0c4cee0bb1e"
+      (reference "#PWR0101") (unit 1) (value "GND") (footprint "")
+    )
     (path "/d96d2f82-dc2a-44d4-a289-0118ed77d142"
       (reference "#PWR0106") (unit 1) (value "GND") (footprint "")
@@
       (reference "BT1") (unit 1) (value "Battery_Cell") (footprint "Connector_JST:JST_PH_S2B-PH-K_1x02_P2.00mm_Horizontal")
     )
+    (path "/ecbed28c-4bdf-4d49-9b6d-4ed18b8a0b0e"
+      (reference "BT2") (unit 1) (value "Conn_01x02") (footprint "Connector_PinHeader_2.54mm:PinHeader_1x02_P2.54mm_Vertical")
+    )
     (path "/e41759dc-e8b4-4683-8ab7-83c4b7632e4d"
