File: mykeeb/rev2/pcb/mykeeb.kicad_sch (KiCad schematic)
At the start: 104 parts, among them K0 KEYSW, K1 KEYSW, K10 KEYSW, K11 KEYSW, K12 KEYSW, K13 KEYSW, K14 KEYSW, K15 KEYSW, K2 KEYSW, K20 KEYSW, K21 KEYSW, K22 KEYSW, K23 KEYSW, K24 KEYSW, K25 KEYSW, K3 KEYSW, K30 KEYSW, K31 KEYSW, K32 KEYSW, K33 KEYSW, K34 KEYSW, K35 KEYSW, K4 KEYSW, K42 KEYSW, K43 KEYSW, K45 KEYSW, K5 KEYSW, K6 KEYSW, SW1 SW_Push, U1 ProMicro

Commit message: wip
Signed-off-by: Maximilian Huber <gh@maxhbr.de>
Parts:
- removed D36: DIODE, Keebio-Parts:D_SOD123F, symbol pspice:DIODE
- removed JPbat+a0, JPbat+b0, JPc0a1, JPc0b1, JPc1a1, JPc1b1, JPc2a1, JPc2b1, JPc3a1, JPc3b1, JPc4a1, JPc4b1, JPc5a1, JPc5b1, JPc6a1, JPc6b1, JPgbda0, JPgndb0, JPr0a1, JPr0b1, JPr1a1, JPr1b1, JPr2a1, JPr2b1, JPr3a1, JPr3b1, JPr4a1, JPr4b1, JPresa0, JPresb0: SolderJumper_2_Open, Jumper:SolderJumper-2_P1.3mm_Open_TrianglePad1.0x1.5mm, symbol Jumper:SolderJumper_2_Open
- removed K36: (no value), symbol keyboard_parts:KEYSW
- added D40, D41: DIODE, mykeeb:my_dual_D_SOD123F_v2, symbol pspice:DIODE
- added K40, K41: KEYSW, mykeeb:Kailh_socket_MX_reversible_1u, symbol keyboard_parts:KEYSW
- D0: value (none) -> DIODE; footprint (none) -> mykeeb:my_dual_D_SOD123F_v2
- D1, D10, D11, D12, D13, D14, D15, D16, D2, D20, D21, D22, D23, D24, D25, D26, D3, D30, D31, D32, D33, D34, D35, D4, D42, D43, D44, D45, D46, D5, D6: footprint Keebio-Parts:D_SOD123F -> mykeeb:my_dual_D_SOD123F_v2
- K16: value (none) -> KEYSW; footprint (none) -> mykeeb:Kailh_socket_MX_reversible_1.5u
- K26, K46: value (none) -> KEYSW; footprint (none) -> mykeeb:Kailh_socket_MX_reversible_1u
- K42, K45: value KEYSW -> (none); footprint mykeeb:Kailh_socket_MX_reversible_1u -> (none)
- U1: value ProMicro -> (none); footprint Keebio-Parts:ArduinoProMicro-BackSide -> (none)
Connections:
- net b0a is gone; now on net Bat+: U1.24 (RAW)
- net c0a is gone; now on net col0: U1.19 (A2/PF5)
- net c1a is gone; now on net col1: U1.18 (A1/PF6)
- net c2a is gone; now on net col2: U1.17 (A0/PF7)
- net c2b is gone; now on net row0: U1.8 (5/PC6)
- net c3a is gone; now on net col3: U1.16 (15/PB1)
- net c3b is gone; now on net row1: U1.9 (6/PD7)
- net c4a is gone; now on net col4: U1.15 (14/PB3)
- net c4b is gone; now on net row2: U1.10 (7/PE6)
- net c5a is gone; now on net col5: U1.14 (16/PB2)
- net c5b is gone; now on net row3: U1.11 (8/PB4)
- net c6a is gone; now on net col6: U1.13 (10/PB6)
- net c6b is gone; now on net row4: U1.12 (9/PB5)
- net g0a is gone; now on net GND: U1.23 (GND)
- net rst0a is gone; now on net RST: U1.22 (RST)
- net rst0b is gone; now on net GND: U1.3 (GND)
- net GND: now also U1.4 (GND)
- net col0: now also K40.1
- net col1: now also K41.1
- net row4: now also D40.2 (A), D41.2 (A)
- net b0b: no longer names the net of U1.1 (TX0/PD3)
- net c0b: no longer names the net of U1.6 (3/PD0)
- net c1b: no longer names the net of U1.7 (4/PD4)
- net g0b: no longer names the net of U1.2 (RX1/PD2)
- new net: D40.1 (K), K40.2
- new net: D41.1 (K), K41.2
- no-connect marks 6 -> 9
Other:
- moved on the sheet: BT1, D0, D1, D10, D11, D12, D13, D14, D15, D16, D2, D20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
