File: mykeeb/rev3/pcb/mykeeb.kicad_pcb (KiCad board)
At the start: 2 copper layers, 158.4 x 94.1 mm, 74 parts, among them J1 Conn_02x08_Odd_Even, K0 KEYSW, K1 KEYSW, K10 KEYSW, K11 KEYSW, K12 KEYSW, K13 KEYSW, K14 KEYSW, K15 KEYSW, K16 KEYSW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

Commit message: wip on rev3
Signed-off-by: Maximilian Huber <gh@maxhbr.de>
Parts:
- added H10: Hole, mykeeb:breakaway-hole, F.Cu at (82.2, 103.6)
- added H11: Hole, mykeeb:breakaway-hole, F.Cu at (141.7, 103.6)
- added H12: Hole, mykeeb:breakaway-hole, F.Cu at (145.3, 101.2)
- added H13: Hole, mykeeb:breakaway-hole, F.Cu at (147.6, 101.2)
- added H14: Hole, mykeeb:breakaway-hole, F.Cu at (139.3, 103.6)
- added H15: Hole, mykeeb:breakaway-hole, F.Cu at (79.8, 103.6)
- added H16: Hole, mykeeb:breakaway-hole, F.Cu at (147.6, 103.6)
- added H17: Hole, mykeeb:breakaway-hole, F.Cu at (88.1, 101.2)
- added H18: Hole, mykeeb:breakaway-hole, F.Cu at (139.3, 101.2)
- added H19: Hole, mykeeb:breakaway-hole, F.Cu at (141.7, 101.2)
- added H20: Hole, mykeeb:breakaway-hole, F.Cu at (85.7, 103.6)
- added H21: Hole, mykeeb:breakaway-hole, F.Cu at (88.1, 103.6)
- added H22: Hole, mykeeb:breakaway-hole, F.Cu at (85.7, 101.2)
- added H23: Hole, mykeeb:breakaway-hole, F.Cu at (86.9, 103.6)
- added H24: Hole, mykeeb:breakaway-hole, F.Cu at (81.0, 101.2)
- added H25: Hole, mykeeb:breakaway-hole, F.Cu at (140.5, 101.2)
- added H26: Hole, mykeeb:breakaway-hole, F.Cu at (140.5, 103.6)
- added H27: Hole, mykeeb:breakaway-hole, F.Cu at (146.4, 103.6)
- added H28: Hole, mykeeb:breakaway-hole, F.Cu at (86.9, 101.2)
- added H29: Hole, mykeeb:breakaway-hole, F.Cu at (146.4, 101.2)
- added H30: Hole, mykeeb:breakaway-hole, F.Cu at (81.0, 103.6)
- added H5: MountingHole, MountingHole:MountingHole_3.2mm_M3, F.Cu at (135.7, 113.1)
- added H6: MountingHole, MountingHole:MountingHole_3.2mm_M3, F.Cu at (75.0, 111.9)
- added H7: Hole, mykeeb:breakaway-hole, F.Cu at (82.2, 101.2)
- added H8: Hole, mykeeb:breakaway-hole, F.Cu at (79.8, 101.2)
- added H9: Hole, mykeeb:breakaway-hole, F.Cu at (145.3, 103.6)
- added K40: KEYSW, mykeeb:Kailh_socket_MX_reversible_1u, F.Cu at (65.5, 121.4)
- added K41: KEYSW, mykeeb:Kailh_socket_MX_reversible_1u, F.Cu at (87.9, 114.1)
- added K42: KEYSW, mykeeb:Kailh_socket_MX_reversible_1.25u, F.Cu at (111.9, 117.9)
- added K43: KEYSW, mykeeb:Kailh_socket_MX_reversible_1u, F.Cu at (134.9, 127.2)
- added K44: KEYSW, mykeeb:Kailh_socket_MX_reversible_1u, F.Cu at (151.7, 141.8)
- added K45: KEYSW, mykeeb:Kailh_socket_MX_reversible_1u, F.Cu at (165.7, 127.8)
- added K46: KEYSW, mykeeb:Kailh_socket_MX_reversible_1u, F.Cu at (151.7, 113.8)
Routing:
- net row4: track 33.5 -> 298.6 mm, vias 1 -> 8
- net Net-(D43-Pad2): track 2.92 -> 173.6 mm, vias 0 -> 1
- net Net-(D40-Pad2): track 2.92 -> 163.1 mm, vias 0 -> 1
- net Net-(D42-Pad2): track 2.92 -> 151.9 mm, vias 0 -> 1
- net Net-(D41-Pad2): track 2.92 -> 137.9 mm, vias 0 -> 1
- net Net-(D45-Pad2): track 2.92 -> 111.0 mm, vias 0 -> 1
- net Net-(D44-Pad2): track 2.92 -> 106.7 mm, vias 0 -> 1
- net Net-(D46-Pad2): track 2.92 -> 81.1 mm, vias 0 -> 1
- net GND: track 81.5 -> 102.6 mm, vias 12 -> 31
- net row2: track 193.3 -> 199.0 mm, vias 4 -> 3
- net col6: track 189.3 -> 188.0 mm, vias 5 -> 6
- net row3: vias 4 -> 2
Other:
- board size 158.4 x 94.1 mm -> 161.9 x 134.5 mm

Commit message: wip on rev3
Signed-off-by: Maximilian Huber <gh@maxhbr.de>
Parts:
- added H31: MountingHole, MountingHole:MountingHole_3.2mm_M3, F.Cu at (151.8, 128.0)
- added J11: Conn_01x05, Connector_PinSocket_2.54mm:PinSocket_1x05_P2.54mm_Vertical, B.Cu at (135.9, 34.8)
- added J2: Conn_01x02, Connector_PinSocket_2.54mm:PinSocket_1x02_P2.54mm_Vertical, B.Cu at (164.4, 33.4)
- added J3: Conn_01x02, Connector_PinHeader_1.27mm:PinHeader_1x02_P1.27mm_Vertical, B.Cu at (81.6, 105.4)
- added J4: Conn_01x02, Connector_PinHeader_1.27mm:PinHeader_1x02_P1.27mm_Vertical, B.Cu at (87.5, 105.4)
- added J5: Conn_01x02, Connector_PinHeader_1.27mm:PinHeader_1x02_P1.27mm_Vertical, B.Cu at (141.1, 105.4)
- added J6: Conn_01x02, Connector_PinHeader_1.27mm:PinHeader_1x02_P1.27mm_Vertical, B.Cu at (147.0, 105.4)
- H23, H24, H25, H26, H27, H28, H29, H30: footprint mykeeb:breakaway-hole -> mykeeb:breakaway-hole-center
- moved H6 1.19 mm to (75.0, 110.7)
Connections:
- U1 pad 21: unconnected-(U1-Pad21) -> VCC
- U1 pad 5: unconnected-(U1-Pad5) -> SDA
- U1 pad 6: unconnected-(U1-Pad6) -> SCL
Routing:
- net SCL: track 0.00 -> 31.1 mm, vias 0 -> 1
- net SDA: track 0.00 -> 27.2 mm, vias 0 -> 1
- net VCC: track 0.00 -> 27.0 mm, vias 0 -> 1
- net GND: track 102.6 -> 126.1 mm, vias 31 -> 34
- net unconnected-(U1-Pad21): track 9.49 -> 0.00 mm, vias 1 -> 0
- net unconnected-(U1-Pad6): track 9.49 -> 0.00 mm, vias 1 -> 0
- net unconnected-(U1-Pad5): track 9.49 -> 0.00 mm, vias 1 -> 0
- net col6: track 188.0 -> 192.4 mm
- net Net-(D41-Pad2): track 137.9 -> 136.4 mm
- net Net-(D42-Pad2): track 151.9 -> 152.7 mm
Other:
- outline, holes or cut-outs redrawn
- board text added: "+"
- board text added: "github.com/maxhbr"

Commit message: rev3
Signed-off-by: Maximilian Huber <gh@maxhbr.de>
Routing:
- net row4: track 298.9 -> 297.9 mm
- net VCC: track 27.0 -> 26.0 mm
- net GND: vias 34 -> 35
Changed lines of the file:
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@@
     (effects (font (size 1 1) (thickness 0.15)) (justify mirror))
   )
-  (gr_text "+" (at 166.092327 31.551589) (layer "B.SilkS")
+  (gr_text "+" (at 164.306285 35.718739 180) (layer "B.SilkS")
     (effects (font (size 3 3) (thickness 0.15)) (justify mirror))
   )
@@
     (effects (font (size 3 3) (thickness 0.15)) (justify mirror))
   )
-  (gr_text "+" (at 166.092327 31.551589) (layer "F.SilkS")
+  (gr_text "+" (at 164.306285 35.718739 180) (layer "F.SilkS")
     (effects (font (size 3 3) (thickness 0.15)))
   )
@@
   (segment locked (start 92.56825 53.277625) (end 96.440625 57.15) (width 0.25) (layer "F.Cu") (net 5))
   (segment locked (start 91.678125 53.277625) (end 92.56825 53.277625) (width 0.25) (layer "F.Cu") (net 5))
-  (segment locked (start 149.411295 55.177295) (end 149.411295 55.118) (width 0.25) (layer "F.Cu") (net 5))
   (segment locked (start 141.684375 77.422375) (end 141.986 77.724) (width 0.25) (layer "F.Cu") (net 5))
   (segment locked (start 160.2 46.736) (end 160.962 45.974) (width 0.25) (layer "F.Cu") (net 5))
@@
   (segment locked (start 58.340625 80.9625) (end 70.246875 80.9625) (width 0.25) (layer "F.Cu") (net 6))
   (segment locked (start 159.288 49.276) (end 160.2 49.276) (width 0.25) (layer "F.Cu") (net 6))
-  (segment locked (start 72.628125 78.58125) (end 72.628125 78.28075) (width 0.25) (layer "F.Cu") (net 6))
   (segment locked (start 126.20625 84.534375) (end 127.396875 84.534375) (width 0.25) (layer "F.Cu") (net 6))
   (segment locked (start 135.454354 81.912536) (end 135.639 81.72789) (width 0.25) (layer "F.Cu") (net 6))
@@
   (segment locked (start 141.826698 131.572) (end 142.494 131.572) (width 0.25) (layer "B.Cu") (net 8))
   (segment locked (start 73.301527 119.863455) (end 71.882 118.443928) (width 0.25) (layer "B.Cu") (net 8))
+  (segment locked (start 168.146 54.356) (end 168.146 59.199) (width 0.25) (layer "B.Cu") (net 8))
   (segment locked (start 118.563749 122.281999) (end 120.449748 120.396) (width 0.25) (layer "B.Cu") (net 8))
   (segment locked (start 160.962 53.594) (end 166.55 53.594) (width 0.25) (layer "B.Cu") (net 8))
   (segment locked (start 116.131748 124.714) (end 103.460875 124.714) (width 0.25) (layer "B.Cu") (net 8))
   (segment locked (start 170.546175 133.604) (end 169.242275 134.9079) (width 0.25) (layer "B.Cu") (net 8))
-  (segment locked (start 168.146 54.356) (end 168.146 54.546614) (width 0.25) (layer "B.Cu") (net 8))
   (segment locked (start 103.460875 124.714) (end 95.428125 116.68125) (width 0.25) (layer "B.Cu") (net 8))
-  (segment locked (start 163.591 59.101614) (end 163.591 61.214) (width 0.25) (layer "B.Cu") (net 8))
   (segment locked (start 95.428125 116.68125) (end 89.935375 122.174) (width 0.25) (layer "B.Cu") (net 8))
   (segment locked (start 140.180868 140.688868) (end 140.180868 133.21783) (width 0.25) (layer "B.Cu") (net 8))
@@
   (segment locked (start 155.242275 148.9079) (end 148.3999 148.9079) (width 0.25) (layer "B.Cu") (net 8))
   (segment locked (start 167.312 54.356) (end 168.146 54.356) (width 0.25) (layer "B.Cu") (net 8))
+  (segment locked (start 168.146 59.199) (end 166.131 61.214) (width 0.25) (layer "B.Cu") (net 8))
   (segment locked (start 157.734 109.116069) (end 158.834377 110.216446) (width 0.25) (layer "B.Cu") (net 8))
   (segment locked (start 75.612072 122.174) (end 73.301527 119.863455) (width 0.25) (layer "B.Cu") (net 8))
   (segment locked (start 95.428125 114.883875) (end 96.266 114.046) (width 0.25) (layer "B.Cu") (net 8))
   (segment locked (start 71.882 118.443928) (end 71.882 117.602) (width 0.25) (layer "B.Cu") (net 8))
-  (segment locked (start 168.146 54.546614) (end 163.591 59.101614) (width 0.25) (layer "B.Cu") (net 8))
   (segment locked (start 171.704 133.604) (end 170.546175 133.604) (width 0.25) (layer "B.Cu") (net 8))
   (segment locked (start 140.180868 133.21783) (end 138.016698 135.382) (width 0.25) (layer "B.Cu") (net 8))
@@
   (segment locked (start 164.72904 54.39896) (end 166.55 52.578) (width 0.25) (layer "F.Cu") (net 14))
   (segment locked (start 116.344375 72.310625) (end 119.440815 69.214185) (width 0.25) (layer "F.Cu") (net 14))
-  (segment locked (start 123.667065 69.214185) (end 123.825 69.214185) (width 0.25) (layer "F.Cu") (net 14))
   (segment locked (start 149.042585 80.82885) (end 135.990887 80.82885) (width 0.25) (layer "F.Cu") (net 14))
   (segment locked (start 131.793886 76.631849) (end 131.793886 73.453261) (width 0.25) (layer "F.Cu") (net 14))
@@
   (segment locked (start 152.557935 77.949216) (end 152.557935 77.058065) (width 0.25) (layer "F.Cu") (net 15))
   (segment locked (start 135.804689 81.27837) (end 135.442465 80.916146) (width 0.25) (layer "F.Cu") (net 15))
-  (segment locked (start 135.394375 86.598125) (end 135.419375 86.598125) (width 0.25) (layer "F.Cu") (net 15))
   (segment locked (start 152.691489 60.405897) (end 153.953786 59.1436) (width 0.25) (layer "F.Cu") (net 15))
   (via locked (at 153.162 76.454) (size 0.8) (drill 0.4) (layers "F.Cu" "B.Cu") (net 15))
@@
   (segment locked (start 138.1125 91.678125) (end 138.1125 94.04) (width 0.25) (layer "B.Cu") (net 15))
   (segment locked (start 156.08 69.472) (end 155.956 69.472) (width 0.25) (layer "B.Cu") (net 15))
-  (segment locked (start 136.619796 61.560204) (end 136.604375 61.575625) (width 0.25) (layer "B.Cu") (net 15))
   (segment locked (start 160.2 54.356) (end 160.962 55.118) (width 0.25) (layer "B.Cu") (net 15))
   (segment locked (start 159.286 54.356) (end 160.2 54.356) (width 0.25) (layer "B.Cu") (net 15))
@@
   (segment locked (start 173.736 69.43725) (end 172.418375 68.119625) (width 0.25) (layer "B.Cu") (net 15))
   (segment locked (start 134.729854 80.916146) (end 134.729854 96.093604) (width 0.25) (layer "B.Cu") (net 15))
-  (segment locked (start 135.394375 96.758125) (end 135.378954 96.773546) (width 0.25) (layer "B.Cu") (net 15))
   (segment locked (start 135.394375 60.365625) (end 136.604375 61.575625) (width 0.25) (layer "B.Cu") (net 15))
-  (segment locked (start 134.978125 48.974375) (end 134.962704 48.989796) (width 0.25) (layer "B.Cu") (net 15))
   (segment locked (start 134.729854 96.093604) (end 135.394375 96.758125) (width 0.25) (layer "B.Cu") (net 15))
-  (segment locked (start 136.604375 61.575625) (end 136.588954 61.560204) (width 0.25) (layer "B.Cu") (net 15))
   (segment locked (start 170.114369 73.093631) (end 173.736 69.472) (width 0.25) (layer "B.Cu") (net 15))
   (segment locked (start 134.729854 63.450146) (end 134.729854 80.916146) (width 0.25) (layer "B.Cu") (net 15))
-  (segment locked (start 135.394375 49.133125) (end 135.378954 49.148546) (width 0.25) (layer "B.Cu") (net 15))
   (segment locked (start 160.962 55.118) (end 166.55 55.118) (width 0.25) (layer "B.Cu") (net 15))
   (segment locked (start 138.1125 44.053125) (end 138.1125 46.415) (width 0.25) (layer "B.Cu") (net 15))
@@
   (segment locked (start 157.432375 68.119625) (end 156.08 69.472) (width 0.25) (layer "B.Cu") (net 15))
   (segment locked (start 139.3225 64.29375) (end 136.604375 61.575625) (width 0.25) (layer "B.Cu") (net 15))
-  (segment locked (start 135.378954 49.117704) (end 135.394375 49.133125) (width 0.25) (layer "B.Cu") (net 15))
   (segment locked (start 172.418375 68.119625) (end 157.432375 68.119625) (width 0.25) (layer "B.Cu") (net 15))
   (segment locked (start 138.1125 94.04) (end 135.394375 96.758125) (width 0.25) (layer "B.Cu") (net 15))
@@
   (via locked (at 142.279807 85.129759) (size 0.8) (drill 0.4) (layers "F.Cu" "B.Cu") (free) (net 16))
   (via locked (at 165.354 27.94) (size 0.8) (drill 0.4) (layers "F.Cu" "B.Cu") (net 16))
+  (via locked (at 166.687537 58.340633) (size 0.8) (drill 0.4) (layers "F.Cu" "B.Cu") (free) (net 16))
   (via locked (at 75.009375 64.29375) (size 0.8) (drill 0.4) (layers "F.Cu" "B.Cu") (free) (net 16))
   (via locked (at 173.236083 72.032873) (size 0.8) (drill 0.4) (layers "F.Cu" "B.Cu") (free) (net 16))
@@
   (segment locked (start 146.304 118.872) (end 147.903074 118.872) (width 0.25) (layer "B.Cu") (net 56))
   (segment locked (start 147.903074 118.872) (end 150.837 121.805926) (width 0.25) (layer "B.Cu") (net 56))
-  (segment locked (start 146.08 34.823) (end 146.493811 35.236811) (width 0.25) (layer "F.Cu") (net 57))
   (segment locked (start 167.386112 34.036) (end 168.148 34.036) (width 0.25) (layer "F.Cu") (net 57))
-  (segment locked (start 164.365762 33.754238) (end 164.365762 33.362528) (width 0.25) (layer "F.Cu") (net 57))
   (segment locked (start 167.282953 33.932841) (end 166.417794 34.798) (width 0.6) (layer "F.Cu") (net 57))
   (segment locked (start 166.417794 34.798) (end 165.608 34.798) (width 0.6) (layer "F.Cu") (net 57))
@@
         (xy 17.859375 39.290625)
         (xy 19.05 38.1)
-        (xy 42.8625 38.1)
-        (xy 46.434375 34.528125)
+        (xy 44.053059 38.099991)
+        (xy 46.434375 35.718739)
         (xy 46.434375 32.146875)
         (xy 50.00625 28.575)
@@
         (xy 17.859375 39.290625)
         (xy 19.05 38.1)
-        (xy 42.8625 38.1)
-        (xy 46.434375 34.528125)
+        (xy 44.053059 38.099991)
+        (xy 46.434375 35.718739)
         (xy 46.434375 32.146875)
         (xy 50.00625 28.575)
