File: mykeeb/rev3/pcb/mykeeb.kicad_sch (KiCad schematic)
At the start: 74 parts, among them K0 KEYSW, K1 KEYSW, K10 KEYSW, K11 KEYSW, K12 KEYSW, K13 KEYSW, K14 KEYSW, K15 KEYSW, K16 KEYSW, K2 KEYSW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

Commit message: wip on rev3
Signed-off-by: Maximilian Huber <gh@maxhbr.de>
Parts:
- added H10, H11, H12, H13, H14, H15, H16, H17, H18, H20, H21, H22, H7, H8, H9: Hole, mykeeb:breakaway-hole, symbol keebio:Hole
- added H19: (no value), symbol keebio:Hole
- added H5, H6: MountingHole, MountingHole:MountingHole_3.2mm_M3, symbol Mechanical:MountingHole
- added K40, K41, K43, K44, K45, K46: KEYSW, mykeeb:Kailh_socket_MX_reversible_1u, symbol keyboard_parts:KEYSW
- added K42: (no value), symbol keyboard_parts:KEYSW
Connections:
- net row4: now also K40.2, K41.2, K42.2, K43.2, K44.2, K45.2, K46.2
- net at D46.2 (A), J1.16 (Pin_16): now also K46.1
- net at D40.2 (A), J1.4 (Pin_4): now also K40.1
- net at D42.2 (A), J1.8 (Pin_8): now also K42.1
- net at D43.2 (A), J1.10 (Pin_10): now also K43.1
- net at D44.2 (A), J1.12 (Pin_12): now also K44.1
- net at D45.2 (A), J1.14 (Pin_14): now also K45.1
- net at D41.2 (A), J1.6 (Pin_6): now also K41.1
Other:
- moved on the sheet: D0, D1, D10, D11, D12, D13, D14, D15, D16, D2, D20, D21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

Commit message: wip on rev3
Signed-off-by: Maximilian Huber <gh@maxhbr.de>
Parts:
- added H23, H24, H25, H26, H27, H28, H29, H30: (no value), symbol keebio:Hole
- added J11: (no value), symbol Connector_Generic:Conn_01x05
- added J2, J6: (no value), symbol Connector_Generic:Conn_01x02
- added J3, J4, J5: Conn_01x02, Connector_PinHeader_1.27mm:PinHeader_1x02_P1.27mm_Vertical, symbol Connector_Generic:Conn_01x02
Connections:
- net GND: now also J11.1 (Pin_1), J11.2 (Pin_2), J2.2 (Pin_2)
- net row4: now also J6.1 (Pin_1)
- net at D46.2 (A), J1.16 (Pin_16), K46.1: now also J6.2 (Pin_2)
- net VCC: now reaches U1.21 (VCC)
- net VCC: now also J11.5 (Pin_5), J2.1 (Pin_1)
- net SDA: now reaches U1.5 (2/PD1)
- net SDA: now also J11.4 (Pin_4)
- net SCL: now reaches U1.6 (3/PD0)
- net SCL: now also J11.3 (Pin_3)
- net at D40.2 (A), J1.4 (Pin_4), K40.1: now also J3.2 (Pin_2)
- net at D42.2 (A), J1.8 (Pin_8), K42.1: now also J4.2 (Pin_2)
- net at D43.2 (A), J1.10 (Pin_10), K43.1: now also J4.1 (Pin_1)
- net at D44.2 (A), J1.12 (Pin_12), K44.1: now also J5.2 (Pin_2)
- net at D45.2 (A), J1.14 (Pin_14), K45.1: now also J5.1 (Pin_1)
- net at D41.2 (A), J1.6 (Pin_6), K41.1: now also J3.1 (Pin_1)
- no-connect marks 8 -> 5
Other:
- moved on the sheet: BT1, FID1, FID2, FID3, H1, H10, H11, H12, H13, H14, H15, H16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

Commit message: rev3
Signed-off-by: Maximilian Huber <gh@maxhbr.de>
Parts:
- added H31: MountingHole, MountingHole:MountingHole_3.2mm_M3, symbol Mechanical:MountingHole
Changed lines of the file:
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@@
     (pin "2")
+  )
+  (symbol (lib_id "Mechanical:MountingHole") (at 387.35 191.77 0) (unit 1)
+    (in_bom yes) (on_board yes) (fields_autoplaced)
+    (property "Reference" "H31" (id 0) (at 389.89 190.4999 0)
+      (effects (font (size 1.27 1.27)) (justify left))
+    )
+    (property "Value" "MountingHole" (id 1) (at 389.89 193.0399 0)
+      (effects (font (size 1.27 1.27)) (justify left))
+    )
+    (property "Footprint" "MountingHole:MountingHole_3.2mm_M3" (id 2) (at 387.35 191.77 0)
+      (effects (font (size 1.27 1.27)) hide)
+    )
+    (property "Datasheet" "~" (id 3) (at 387.35 191.77 0)
+      (effects (font (size 1.27 1.27)) hide)
+    )
   )
   (symbol (lib_id "keebio:ProMicro") (at 57.15 41.91 0) (unit 1)
@@
       (reference "H30") (unit 1) (value "Hole") (footprint "mykeeb:breakaway-hole-center")
     )
+    (path "/207bc95f-5d5d-4eff-b3a7-9d02aec97b29"
+      (reference "H31") (unit 1) (value "MountingHole") (footprint "MountingHole:MountingHole_3.2mm_M3")
+    )
     (path "/4c97b8e7-b85d-4d19-880f-480e666b3f54"
