File: mykeeb/rev4b/pcb/mykeeb.kicad_pcb (KiCad board)
At the start: 2 copper layers, 180.4 x 135.1 mm, 100 parts, among them J1 Conn_02x07_Odd_Even, J11 Conn_01x05, J2 Conn_01x02, J3 Conn_02x07_Odd_Even, J4 Conn_02x07_Odd_Even, J7 Conn_02x07_Odd_Even, K0 KEYSW, K1 KEYSW, K10 KEYSW, K11 KEYSW, K12 KEYSW, K13 KEYSW, K14 KEYSW, K15 KEYSW, K16 KEYSW, K2 KEYSW, K20 KEYSW, K21 KEYSW, K22 KEYSW, K23 KEYSW, K24 KEYSW, K25 KEYSW, K26 KEYSW, K3 KEYSW, K30 KEYSW, K31 KEYSW, K32 KEYSW, K33 KEYSW, K34 KEYSW, K35 KEYSW, K4 KEYSW, K40 KEYSW, K41 KEYSW, K42 KEYSW, K43 KEYSW, K44 KEYSW, K45 KEYSW, K46 KEYSW, K5 KEYSW, K6 KEYSW, SW1 SW_Push, SW36 SW_Push, U1 ProMicro

Commit message: rev4b
Signed-off-by: Maximilian Huber <gh@maxhbr.de>
Parts:
- removed BT1: Battery_Cell, Connector_JST:JST_PH_S2B-PH-K_1x02_P2.00mm_Horizontal
- removed D40, D41, D42, D43, D44, D45, D46: DIODE, mykeeb:my_dual_D_SOD123F_v2b
- removed H10, H11, H12, H13, H14, H15, H16, H7, H8, H9: Hole, mykeeb:breakaway
- removed H31, H5, H6: MountingHole, MountingHole:MountingHole_3.2mm_M3
- removed J1, J3, J4, J7: Conn_02x07_Odd_Even, Connector_PinHeader_2.54mm:PinHeader_2x07_P2.54mm_Vertical
- removed J11: Conn_01x05, Connector_PinSocket_2.54mm:PinSocket_1x05_P2.54mm_Vertical
- removed K40, K41, K43, K44, K45, K46: KEYSW, mykeeb:Kailh_socket_MX_reversible_1u
- removed K42: KEYSW, mykeeb:Kailh_socket_MX_reversible_1.25u
- removed SW1: SW_Push, Button_Switch_THT:SW_PUSH_6mm
- removed U1: ProMicro, mykeeb:my_reversible_Pro_Micro
- J2: value Conn_01x02 -> Conn_01x16_Male; footprint Connector_PinHeader_2.54mm:PinHeader_1x02_P2.54mm_Vertical -> mykeeb:adapterBoard; moved to F.Cu
- SW36: footprint Button_Switch_THT:SW_PUSH_6mm -> Button_Switch_THT:SW_PUSH_6mm_H7.3mm
- SWbat1: moved to B.Cu
- moved J2 84.6 mm to (94.1, 58.3)
- moved SWbat1 79.7 mm to (120.1, 28.6)
- moved H4 31.6 mm to (155.4, 64.9)
- moved SW36 28.6 mm to (157.6, 52.7)
- moved D36 28.6 mm to (151.8, 54.8)
- moved FID2 13.9 mm to (133.4, 57.7)
- moved H3 0.60 mm to (136.9, 30.4)
Connections:
- J2 pad 1: VCC -> col0b
- J2 pad 2: GND -> col1b
- SWbat1 pad 1: Net-(BT1-Pad1) -> unconnected-(SWbat1-Pad1)
- SWbat1 pad 2: Bat+ -> Net-(J2-Pad13)
- SWbat1 pad 3: unconnected-(SWbat1-Pad3) -> Net-(J2-Pad14)
Routing:
- net Net-(K42-Pad2): track 215.9 -> 0.00 mm, vias 7 -> 0
- net Net-(K40-Pad1): track 132.9 -> 0.00 mm, vias 2 -> 0
- net GND: track 106.2 -> 0.00 mm, vias 8 -> 0
- net Net-(K41-Pad1): track 104.6 -> 0.00 mm, vias 1 -> 0
- net col2b: track 226.3 -> 124.6 mm
- net col0b: track 274.3 -> 173.3 mm
- net col1b: track 253.1 -> 153.2 mm
- net col3b: track 210.2 -> 113.5 mm
- net Net-(K42-Pad1): track 82.3 -> 0.00 mm, vias 1 -> 0
- net col4b: track 190.1 -> 126.1 mm
- net Net-(K43-Pad1): track 63.8 -> 0.00 mm, vias 2 -> 0
- net col5b: track 173.3 -> 118.4 mm
- net col0: track 53.0 -> 0.00 mm, vias 1 -> 0
- net Net-(J2-Pad14): track 0.00 -> 49.5 mm, vias 0 -> 5
- net Net-(K44-Pad1): track 48.7 -> 0.00 mm, vias 1 -> 0
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- added copper zone on B.Cu, net gndb
- added copper zone on F.Cu, net gndb
- removed copper zone on B.Cu, net GND
- removed copper zone on F.Cu, net GND
Other:
- board size 180.4 x 135.1 mm -> 141.7 x 94.1 mm
