File: mykeeb/rev4b/pcb/mykeeb.kicad_sch (KiCad schematic)
At the start: 100 parts, among them J1 Conn_02x07_Odd_Even, J11 Conn_01x05, J3 Conn_02x07_Odd_Even, J4 Conn_02x07_Odd_Even, K0 KEYSW, K1 KEYSW, K10 KEYSW, K11 KEYSW, K12 KEYSW, K13 KEYSW, K14 KEYSW, K15 KEYSW, K16 KEYSW, K2 KEYSW, K20 KEYSW, K21 KEYSW, K22 KEYSW, K23 KEYSW, K24 KEYSW, K25 KEYSW, K26 KEYSW, K3 KEYSW, K30 KEYSW, K31 KEYSW, K32 KEYSW, K33 KEYSW, K34 KEYSW, K35 KEYSW, K4 KEYSW, K40 KEYSW, K41 KEYSW, K42 KEYSW, K43 KEYSW, K44 KEYSW, K45 KEYSW, K46 KEYSW, K5 KEYSW, K6 KEYSW, SW1 SW_Push, SW36 SW_Push, U1 ProMicro

Commit message: rev4b
Signed-off-by: Maximilian Huber <gh@maxhbr.de>
Parts:
- removed BT1: Battery_Cell, Connector_JST:JST_PH_S2B-PH-K_1x02_P2.00mm_Horizontal, symbol Device:Battery_Cell
- removed D40, D41, D42, D43, D44, D45, D46: (no value), symbol pspice:DIODE
- removed H10, H11, H12, H13, H14, H15, H16, H8, H9: Hole, mykeeb:breakaway, symbol keebio:Hole
- removed H31, H5, H6: MountingHole, MountingHole:MountingHole_3.2mm_M3, symbol Mechanical:MountingHole
- removed H7: (no value), symbol keebio:Hole
- removed J1, J3, J4: Conn_02x07_Odd_Even, Connector_PinHeader_2.54mm:PinHeader_2x07_P2.54mm_Vertical, symbol Connector_Generic:Conn_02x07_Odd_Even
- removed J11: Conn_01x05, Connector_PinSocket_2.54mm:PinSocket_1x05_P2.54mm_Vertical, symbol Connector_Generic:Conn_01x05
- removed J2: (no value), symbol Connector_Generic:Conn_01x02
- removed J7: (no value), symbol Connector_Generic:Conn_02x07_Odd_Even
- removed K40, K41, K43, K44, K45, K46: KEYSW, mykeeb:Kailh_socket_MX_reversible_1u, symbol keyboard_parts:KEYSW
- removed K42: KEYSW, mykeeb:Kailh_socket_MX_reversible_1.25u, symbol keyboard_parts:KEYSW
- removed SW1: SW_Push, Button_Switch_THT:SW_PUSH_6mm, symbol Switch:SW_Push
- removed SWbat1: SW_SPST, Connector_PinSocket_2.54mm:PinSocket_1x03_P2.54mm_Vertical, symbol Switch:SW_SPDT
- removed U1: ProMicro, mykeeb:my_reversible_Pro_Micro, symbol keebio:ProMicro
- added J2: (no value), symbol Connector:Conn_01x16_Male
- added SWbat?: SW_SPST, Connector_PinSocket_2.54mm:PinSocket_1x03_P2.54mm_Vertical, symbol Switch:SW_SPDT
- D36: value (none) -> DIODE; footprint (none) -> mykeeb:my_dual_D_SOD123F_v2b
- SW36: footprint Button_Switch_THT:SW_PUSH_6mm -> Button_Switch_THT:SW_PUSH_6mm_H7.3mm
Connections:
- net col0b: now also J2.1 (Pin_1)
- net col1b: now also J2.2 (Pin_2)
- net col2b: now also J2.3 (Pin_3)
- net col3b: now also J2.4 (Pin_4)
- net col4b: now also J2.5 (Pin_5)
- net col5b: now also J2.6 (Pin_6)
- net col6b: now also J2.7 (Pin_7)
- net row0b: now also J2.9 (Pin_9)
- net row1b: now also J2.10 (Pin_10)
- net row2b: now also J2.11 (Pin_11)
- net row3b: now also J2.12 (Pin_12)
- new net: J2.13 (Pin_13), SWbat?.2 (B)
- new net: J2.14 (Pin_14), SWbat?.3 (C)
- new net gndb: J2.16 (Pin_16), J2.8 (Pin_8)
- no-connect marks 5 -> 0
Other:
- moved on the sheet: D0, D1, D10, D11, D12, D13, D14, D15, D16, D2, D20, D21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
