File: PCB/mykeeb_v7a1/mykeeb_v7a1.kicad_sch (KiCad schematic)
At the start: 13 parts, among them SW43 SW_Push, SW44 SW_SPDT, U1 74HC595, U2 xiao-ble

Commit message: update
Signed-off-by: Maximilian Huber <gh@maxhbr.de>
Parts:
- added D1, D10, D11, D12, D13, D14, D15, D2, D3, D4, D5, D6, D7, D8, D9: BAV70, mykeeb:SOT-23, symbol hillside_basic:BAV70_Small
- added D16, D17, D18, D19, D20: D, mykeeb:D3_SMD, symbol Device:D
- added FID1, FID2, FID3: Fiducial, Fiducial:Fiducial_1mm_Mask2mm, symbol Mechanical:Fiducial
- added S0, S1, S10, S11, S12, S13, S14, S15, S16, S2, S20, S21, S22, S23, S24, S25, S26, S3, S30, S31, S32, S33, S34, S35, S36, S4, S40, S41, S42, S43, S44, S45, S46, S5, S6: SW, mykeeb:MX_KAILH_SOCKET_1U, symbol YAEMK:MX_1U
- U2: footprint sepp:xiao-ble-smd-cutout-geist -> pretty:xiao-ble-smd-cutout
Connections:
- new net: D19.2 (A), S36.2
- new net: D20.2 (A), S46.2
- new net: D12.2 (A2), S15.1
- new net: D16.2 (A), S6.2
- new net: D6.1 (A1), S2.2
- new net: D6.2 (A2), S3.1
- new net: D9.2 (A2), S33.1
- new net: D2.2 (A2), S11.1
- new net: D15.1 (A1), S44.2
- new net: D5.1 (A1), S40.2
- new net: D4.1 (A1), S30.2
- new net: D12.1 (A1), S14.2
- new net: D15.2 (A2), S45.1
- new net: D13.1 (A1), S24.2
- new net: D13.2 (A2), S25.1
- new net: D9.1 (A1), S32.2
- new net: D10.1 (A1), S42.2
- new net: D2.1 (A1), S10.2
- new net: D11.1 (A1), S4.2
- new net: D11.2 (A2), S5.1
- new net: D5.2 (A2), S41.1
- new net: D17.2 (A), S16.2
- new net: D8.1 (A1), S22.2
- new net: D8.2 (A2), S23.1
- new net: D14.1 (A1), S34.2
- new net: D14.2 (A2), S35.1
- new net: D18.2 (A), S26.2
- new net: D10.2 (A2), S43.1
- new net: D3.1 (A1), S20.2
- new net: D1.2 (A2), S1.1
- new net: D1.1 (A1), S0.2
- new net: D7.1 (A1), S12.2
- new net: D4.2 (A2), S31.1
- new net: D3.2 (A2), S21.1
- new net: D7.2 (A2), S13.1
- new net col0: S0.1, S10.1, S20.1, S30.1, S40.1
- new net col1: S1.2, S11.2, S21.2, S31.2, S41.2
- new net col2: S12.1, S2.1, S22.1, S32.1, S42.1
- new net col3: S13.2, S23.2, S3.2, S33.2, S43.2
- new net col4: S14.1, S24.1, S34.1, S4.1, S44.1
- new net col5: S15.2, S25.2, S35.2, S45.2, S5.2
- new net col6: S16.1, S26.1, S36.1, S46.1, S6.1
- new net row0: D1.3 (K), D11.3 (K), D16.1 (K), D6.3 (K)
- new net row1: D12.3 (K), D17.1 (K), D2.3 (K), D7.3 (K)
- new net row2: D13.3 (K), D18.1 (K), D3.3 (K), D8.3 (K)
- new net row3: D14.3 (K), D19.1 (K), D4.3 (K), D9.3 (K)
- new net row4: D10.3 (K), D15.3 (K), D20.1 (K), D5.3 (K)
