File: pcb/mykeeb_v7a1.kicad_pcb (KiCad board)
At the start: 2 copper layers, 6.2 x 8.8 mm, 66 parts, among them U1 xiao-ble, U2 74HC595

Commit message: wip
Signed-off-by: Maximilian Huber <gh@maxhbr.de>
Parts:
- removed D10: BAV70, mykeeb:SOT-23
- removed D17, D18: D, mykeeb:D3_SMD
- removed the S41 at (266.6, 161.5)
- removed the S42 at (266.6, 180.6)
- added FID1: Fiducial, Fiducial:Fiducial_1mm_Mask2mm, F.Cu at (345.4, 186.7)
- added FID2: Fiducial, Fiducial:Fiducial_1mm_Mask2mm, F.Cu at (234.0, 162.5)
- added FID3: Fiducial, Fiducial:Fiducial_1mm_Mask2mm, F.Cu at (227.6, 98.6)
- added H9: MountingHole, MountingHole:MountingHole_2.2mm_M2_DIN965, F.Cu at (355.7, 209.0)
- added REF**: mousebites 2mm, TOTEMlib:mousebites_2mm, F.Cu at (207.8, 136.9)
- added REF**: mousebites 2mm, TOTEMlib:mousebites_2mm, F.Cu at (207.8, 106.6)
- added REF**: mousebites 2mm, TOTEMlib:mousebites_2mm, F.Cu at (214.9, 166.1)
- added REF**: mousebites 2mm, TOTEMlib:mousebites_2mm, F.Cu at (207.8, 166.1)
- added REF**: mousebites 2mm, TOTEMlib:mousebites_2mm, F.Cu at (214.9, 136.9)
- added REF**: mousebites 2mm, TOTEMlib:mousebites_2mm, F.Cu at (214.9, 106.6)
- added S45: SW, pretty:MX-1U-Hotswap, F.Cu at (363.1, 217.3)
- added SW_bat1: SW_SPDT, sepp:switch-MSK-12C02-smd, B.Cu at (243.9, 83.7)
- added SW_reset1: SW_Push, sepp:ResetSW, F.Cu at (244.2, 92.9)
- BT1, U2: moved to B.Cu
- D1, D11, D13, D14, D15, D3, D4, D5, D6, D8, D9: footprint mykeeb:SOT-23 -> Package_TO_SOT_SMD:SOT-23; moved to B.Cu
- D12, D2, D7: footprint mykeeb:SOT-23 -> Package_TO_SOT_SMD:SOT-23
- D16, D19, D20: value D -> BAV70; footprint mykeeb:D3_SMD -> Package_TO_SOT_SMD:SOT-23; moved to B.Cu
- S0, S1, S10, S11, S12, S13, S14, S15, S2, S20, S21, S22, S23, S24, S25, S3, S30, S31, S32, S33, S34, S35, S4, S40, S5, S6: footprint mykeeb:MX_KAILH_SOCKET_1U -> pretty:MX-1U-Hotswap
- S36: renamed from S26; footprint mykeeb:MX_KAILH_SOCKET_1U -> pretty:MX-1U-Hotswap
- S37: renamed from S36; footprint mykeeb:MX_KAILH_SOCKET_1U -> pretty:MX-1U-Hotswap
- S41: renamed from S43; footprint mykeeb:MX_KAILH_SOCKET_1U -> pretty:MX-1U-Hotswap
- S42: renamed from S44; footprint mykeeb:MX_KAILH_SOCKET_1U -> pretty:MX-1U-Hotswap
- S43: renamed from S45; footprint mykeeb:MX_KAILH_SOCKET_1U -> pretty:MX-1U-Hotswap
- S44: renamed from S46; footprint mykeeb:MX_KAILH_SOCKET_1U -> pretty:MX-1U-Hotswap
- S7: renamed from S16; footprint mykeeb:MX_KAILH_SOCKET_1U -> pretty:MX-1U-Hotswap
- moved H8 196.5 mm to (361.3, 195.2)
- moved H7 170.2 mm to (318.6, 183.7)
- moved H2 147.3 mm to (235.7, 181.0)
- moved H6 145.2 mm to (331.6, 149.4)
- moved H4 134.4 mm to (273.4, 163.5)
- moved H5 120.6 mm to (328.3, 114.4)
- moved U2 96.3 mm to (286.2, 166.6), turned to -60 degrees
- moved H1 94.3 mm to (234.0, 122.6)
- moved H3 83.7 mm to (253.0, 110.7)
- moved BT1 48.1 mm to (245.1, 97.6), turned to 180 degrees
- moved D16 26.6 mm to (341.1, 127.1)
- moved D19 23.9 mm to (345.6, 178.7), turned to 90 degrees
- moved S40 22.7 mm to (234.0, 191.7)
- moved D15 22.1 mm to (319.9, 176.7)
- moved D5 16.6 mm to (241.3, 180.0)
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Connections:
- D1 pad 1: (no net) -> Net-(D1-A1)
- D1 pad 2: (no net) -> Net-(D1-A2)
- D1 pad 3: (no net) -> row0
- D11 pad 1: (no net) -> Net-(D11-A1)
- D11 pad 2: (no net) -> Net-(D11-A2)
- D11 pad 3: (no net) -> row0
- D12 pad 1: (no net) -> Net-(D12-A1)
- D12 pad 2: (no net) -> Net-(D12-A2)
- D12 pad 3: (no net) -> row1
- D13 pad 1: (no net) -> Net-(D13-A1)
- D13 pad 2: (no net) -> Net-(D13-A2)
- D13 pad 3: (no net) -> row2
- D14 pad 1: (no net) -> Net-(D14-A1)
- D14 pad 2: (no net) -> Net-(D14-A2)
- D14 pad 3: (no net) -> row3
- D15 pad 1: (no net) -> Net-(D15-A1)
- D15 pad 2: (no net) -> Net-(D15-A2)
- D15 pad 3: (no net) -> row4
- D16 pad 1: (no net) -> Net-(D16-A1)
- D16 pad 2: (no net) -> Net-(D16-A2)
- D19 pad 1: (no net) -> Net-(D19-A1)
- D19 pad 2: (no net) -> Net-(D19-A2)
- D2 pad 1: (no net) -> Net-(D2-A1)
- D2 pad 2: (no net) -> Net-(D2-A2)
- D2 pad 3: (no net) -> row1
- D20 pad 1: (no net) -> Net-(D20-A1)
- D20 pad 2: (no net) -> Net-(D20-A2)
- D3 pad 1: (no net) -> Net-(D3-A1)
- D3 pad 2: (no net) -> Net-(D3-A2)
- D3 pad 3: (no net) -> row2
- D4 pad 1: (no net) -> Net-(D4-A1)
- D4 pad 2: (no net) -> Net-(D4-A2)
- D4 pad 3: (no net) -> row3
- D5 pad 1: (no net) -> Net-(D5-A1)
- D5 pad 2: (no net) -> Net-(D5-A2)
- D5 pad 3: (no net) -> row4
- D6 pad 1: (no net) -> Net-(D6-A1)
- D6 pad 2: (no net) -> Net-(D6-A2)
- D6 pad 3: (no net) -> row0
- D7 pad 1: (no net) -> Net-(D7-A1)
- D7 pad 2: (no net) -> Net-(D7-A2)
- D7 pad 3: (no net) -> row1
- D8 pad 1: (no net) -> Net-(D8-A1)
- D8 pad 2: (no net) -> Net-(D8-A2)
- D8 pad 3: (no net) -> row2
- D9 pad 1: (no net) -> Net-(D9-A1)
- D9 pad 2: (no net) -> Net-(D9-A2)
- D9 pad 3: (no net) -> row3
- S0 pad 1: (no net) -> col0
- S0 pad 2: (no net) -> Net-(D1-A1)
- S1 pad 1: (no net) -> Net-(D1-A2)
- S1 pad 2: (no net) -> col1
- S10 pad 1: (no net) -> col0
- S10 pad 2: (no net) -> Net-(D2-A1)
- S11 pad 1: (no net) -> Net-(D2-A2)
- S11 pad 2: (no net) -> col1
- S12 pad 1: (no net) -> col2
- S12 pad 2: (no net) -> Net-(D7-A1)
- S13 pad 1: (no net) -> Net-(D7-A2)
- S13 pad 2: (no net) -> col3
- S14 pad 1: (no net) -> col4
- S14 pad 2: (no net) -> Net-(D12-A1)
- S15 pad 1: (no net) -> Net-(D12-A2)
- S15 pad 2: (no net) -> col5
- S2 pad 1: (no net) -> col2
- S2 pad 2: (no net) -> Net-(D6-A1)
- S20 pad 1: (no net) -> col0
- S20 pad 2: (no net) -> Net-(D3-A1)
- S21 pad 1: (no net) -> Net-(D3-A2)
- S21 pad 2: (no net) -> col1
- S22 pad 1: (no net) -> col2
- S22 pad 2: (no net) -> Net-(D8-A1)
- S23 pad 1: (no net) -> Net-(D8-A2)
- S23 pad 2: (no net) -> col3
- S24 pad 1: (no net) -> col4
- S24 pad 2: (no net) -> Net-(D13-A1)
- S25 pad 1: (no net) -> Net-(D13-A2)
- S25 pad 2: (no net) -> col5
- S3 pad 1: (no net) -> Net-(D6-A2)
- S3 pad 2: (no net) -> col3
- S30 pad 1: (no net) -> col0
- S30 pad 2: (no net) -> Net-(D4-A1)
- S31 pad 1: (no net) -> Net-(D4-A2)
- S31 pad 2: (no net) -> col1
- S32 pad 1: (no net) -> col2
- S32 pad 2: (no net) -> Net-(D9-A1)
- S33 pad 1: (no net) -> Net-(D9-A2)
- S33 pad 2: (no net) -> col3
- S34 pad 1: (no net) -> col4
- S34 pad 2: (no net) -> Net-(D14-A1)
- S35 pad 1: (no net) -> Net-(D14-A2)
- S35 pad 2: (no net) -> col5
- S36 pad 1: (no net) -> col6
- S36 pad 2: (no net) -> Net-(D19-A1)
- S37 pad 1: (no net) -> Net-(D19-A2)
- S37 pad 2: (no net) -> col7
- S4 pad 1: (no net) -> col4
- S4 pad 2: (no net) -> Net-(D11-A1)
- S40 pad 1: (no net) -> col0
- S40 pad 2: (no net) -> Net-(D5-A1)
- S41 pad 1: (no net) -> Net-(D5-A2)
- S41 pad 2: (no net) -> col1
- S42 pad 1: (no net) -> col2
- S42 pad 2: (no net) -> Net-(D15-A1)
- S43 pad 1: (no net) -> Net-(D15-A2)
- S43 pad 2: (no net) -> col3
- S44 pad 1: (no net) -> col4
- S44 pad 2: (no net) -> Net-(D20-A1)
- S5 pad 1: (no net) -> Net-(D11-A2)
- S5 pad 2: (no net) -> col5
- S6 pad 1: (no net) -> col6
- S6 pad 2: (no net) -> Net-(D16-A1)
- S7 pad 1: (no net) -> Net-(D16-A2)
- S7 pad 2: (no net) -> col7
- U2 pad 1: COL5 -> COL1
- U2 pad 15: COL1 -> COL0
- U2 pad 2: COL4 -> COL5
- U2 pad 3: COL3 -> COL4
- U2 pad 4: COL2 -> COL3
- U2 pad 5: COL6 -> COL2
- U2 pad 6: COL7 -> COL6
- U2 pad 7: unconnected-(U2-QH-Pad7) -> COL7
Other:
- board size 6.2 x 8.8 mm -> 326.6 x 145 mm
