File: mykeeb_v7a2/mykeeb_v7a2.kicad_pcb (KiCad board)
At the start: 2 copper layers, 160 x 127.5 mm, 52 parts, among them U1 xiao-ble

Commit message: update
Signed-off-by: Maximilian Huber <gh@maxhbr.de>
Parts:
- added D1: BAV70, Package_TO_SOT_SMD:SOT-23, F.Cu at (161.9, 117.0)
- added D11: BAV70, Package_TO_SOT_SMD:SOT-23, F.Cu at (47.6, 72.6)
- added D12: BAV70, Package_TO_SOT_SMD:SOT-23, F.Cu at (85.7, 108.1)
- added D13: BAV70, Package_TO_SOT_SMD:SOT-23, F.Cu at (85.7, 96.2)
- added D14: BAV70, Package_TO_SOT_SMD:SOT-23, F.Cu at (85.7, 77.4)
- added D15: BAV70, Package_TO_SOT_SMD:SOT-23, F.Cu at (75.6, 61.9)
- added D2: BAV70, Package_TO_SOT_SMD:SOT-23, F.Cu at (161.9, 106.6)
- added D20: BAV70, Package_TO_SOT_SMD:SOT-23, F.Cu at (39.3, 32.7)
- added D3: BAV70, Package_TO_SOT_SMD:SOT-23, F.Cu at (161.9, 88.1)
- added D4: BAV70, Package_TO_SOT_SMD:SOT-23, F.Cu at (161.9, 69.1)
- added D5: BAV70, Package_TO_SOT_SMD:SOT-23, F.Cu at (103.0, 62.5)
- added D6: BAV70, Package_TO_SOT_SMD:SOT-23, F.Cu at (63.1, 114.9)
- added D7: BAV70, Package_TO_SOT_SMD:SOT-23, F.Cu at (123.8, 119.4)
- added D8: BAV70, Package_TO_SOT_SMD:SOT-23, F.Cu at (123.8, 102.4)
- added D9: BAV70, Package_TO_SOT_SMD:SOT-23, F.Cu at (123.8, 83.3)
- added FID1: Fiducial, Fiducial:Fiducial_1mm_Mask2mm, F.Cu at (176.8, 127.9)
- added FID2: Fiducial, Fiducial:Fiducial_1mm_Mask2mm, F.Cu at (32.1, 16.0)
- added FID3: Fiducial, Fiducial:Fiducial_1mm_Mask2mm, F.Cu at (166.1, 44.6)
- added L_BT1: Battery_Cell, Connector_JST:JST_PH_S2B-PH-K_1x02_P2.00mm_Horizontal, B.Cu at (135.9, 134.0)
- added L_S0: SW, pretty:MX-1U-Hotswap, F.Cu at (171.5, 128.0)
- added L_S10: SW, pretty:MX-1U-Hotswap, F.Cu at (172.6, 107.8)
- added L_S11: SW, pretty:MX-1U-Hotswap, F.Cu at (152.4, 108.9)
- added L_S12: SW, pretty:MX-1U-Hotswap, F.Cu at (133.4, 120.8)
- added L_S13: SW, pretty:MX-1U-Hotswap, F.Cu at (114.3, 126.8)
- added L_S14: SW, pretty:MX-1U-Hotswap, F.Cu at (95.3, 119.7)
- added L_S15: SW, pretty:MX-1U-Hotswap, F.Cu at (76.2, 117.3)
- added L_S2: SW, pretty:MX-1U-Hotswap, F.Cu at (57.2, 126.8)
- added L_S20: SW, pretty:MX-1U-Hotswap, F.Cu at (172.6, 88.6)
- added L_S21: SW, pretty:MX-1U-Hotswap, F.Cu at (152.4, 89.9)
- added L_S22: SW, pretty:MX-1U-Hotswap, F.Cu at (133.4, 101.8)
- added L_S23: SW, pretty:MX-1U-Hotswap, F.Cu at (114.3, 107.8)
- added L_S24: SW, pretty:MX-1U-Hotswap, F.Cu at (95.3, 100.6)
- added L_S25: SW, pretty:MX-1U-Hotswap, F.Cu at (76.2, 98.2)
- added L_S3: SW, pretty:MX-1U-Hotswap, F.Cu at (57.2, 103.0)
- added L_S30: SW, pretty:MX-1U-Hotswap, F.Cu at (171.5, 68.5)
- added L_S31: SW, pretty:MX-1U-Hotswap, F.Cu at (152.4, 70.8)
- added L_S32: SW, pretty:MX-1U-Hotswap, F.Cu at (133.4, 82.7)
- added L_S33: SW, pretty:MX-1U-Hotswap, F.Cu at (114.3, 88.7)
- added L_S34: SW, pretty:MX-1U-Hotswap, F.Cu at (95.3, 81.6)
- added L_S35: SW, pretty:MX-1U-Hotswap, F.Cu at (76.2, 79.2)
- added L_S4: SW, pretty:MX-1U-Hotswap, F.Cu at (57.1, 79.2)
- added L_S40: SW, pretty:MX-1U-Hotswap, F.Cu at (161.9, 49.4)
- added L_S42: SW, pretty:MX-1U-Hotswap, F.Cu at (89.3, 60.1)
- added L_S43: SW, pretty:MX-1U-Hotswap, F.Cu at (63.8, 54.1)
- added L_S44: SW, pretty:MX-1U-Hotswap, F.Cu at (46.4, 41.1)
- added L_S5: SW, pretty:MX-1U-Hotswap, F.Cu at (35.4, 59.4)
- added L_SW_bat1: SW_SPDT, sepp:switch-MSK-12C02-smd, B.Cu at (136.9, 141.1)
- added L_SW_reset1: SW_Push, Button_Switch_SMD:SW_SPST_TL3342, B.Cu at (152.4, 131.6)
- added L_U1: xiao-ble, pretty:xiao-ble-smd-cutout, F.Cu at (152.4, 131.1)
- added REF**: breakaway-mousebites, pretty:breakaway-mousebites, F.Cu at (143.5, 149.4)
- added REF**: breakaway-mousebites, pretty:breakaway-mousebites, F.Cu at (58.3, 153.6)
- added REF**: breakaway-mousebites, pretty:breakaway-mousebites, F.Cu at (161.3, 149.4)
- added REF**: breakaway-mousebites, pretty:breakaway-mousebites, F.Cu at (58.3, 141.7)
- added REF**: breakaway-mousebites, pretty:breakaway-mousebites, F.Cu at (161.3, 141.7)
- added REF**: breakaway-mousebites, pretty:breakaway-mousebites, F.Cu at (58.3, 137.5)
- added REF**: breakaway-mousebites, pretty:breakaway-mousebites, F.Cu at (58.3, 149.4)
- added REF**: breakaway-mousebites, pretty:breakaway-mousebites, F.Cu at (143.5, 141.7)
- added locked: SW, pretty:MX-1U-Hotswap, F.Cu at (114.3, 54.1)
- added locked: SW, pretty:MX-1U-Hotswap, F.Cu at (32.7, 23.8)
- FID1, FID2, FID3: moved to B.Cu
- S1: moved to F.Cu
- SW_reset1: footprint pretty:PushSW -> Button_Switch_SMD:SW_SPST_TL3342; moved to B.Cu
- moved FID3 247.1 mm to (166.1, 246.5), turned to 180 degrees
- moved FID2 233.1 mm to (32.1, 275.1), turned to 180 degrees
- moved FID1 198.3 mm to (176.8, 163.2), turned to 180 degrees
- moved locked 193.5 mm to (32.7, 267.3), turned to 60 degrees
- moved S5 189.6 mm to (35.4, 231.7), turned to -143 degrees
- moved S10 188.2 mm to (172.6, 183.3), turned to 85 degrees
- moved S20 188.2 mm to (172.6, 202.5), turned to 85 degrees
- moved S0 186.6 mm to (171.5, 163.1), turned to 90 degrees
- moved S30 186.6 mm to (171.5, 222.6), turned to 90 degrees
- moved D20 184.0 mm to (39.3, 258.4)
- moved S1 180.8 mm to (167.0, 151.8), turned to 0 degrees
- moved S44 174.1 mm to (46.4, 250.0), turned to 45 degrees
- moved D4 173.4 mm to (161.9, 222.1)
- moved D1 173.4 mm to (161.9, 174.1)
- moved D3 173.4 mm to (161.9, 203.0)
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Routing:
- net BAT+: track 31.2 -> 0.00 mm
- net Net-(D1-A2): track 27.0 -> 0.00 mm
- net ROW1: track 0.00 -> 18.6 mm
- net L_ROW1: track 0.00 -> 18.6 mm
- net ROW2: track 0.00 -> 16.4 mm
- net L_ROW2: track 0.00 -> 16.4 mm
- net ROW3: track 0.00 -> 14.7 mm
- net L_ROW3: track 0.00 -> 14.7 mm
- net L_COL3: track 0.00 -> 13.3 mm, vias 0 -> 2
- net COL3: track 0.00 -> 13.3 mm, vias 0 -> 2
- net COL2: track 0.00 -> 12.1 mm, vias 0 -> 2
- net L_COL2: track 0.00 -> 12.1 mm, vias 0 -> 2
- net COL0: track 0.00 -> 11.8 mm
- net COL4: track 0.00 -> 11.7 mm, vias 0 -> 2
- net L_COL4: track 0.00 -> 11.7 mm, vias 0 -> 2
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Other:
- board size 160 x 127.5 mm -> 160.4 x 265.5 mm

Commit message: routing
Signed-off-by: Maximilian Huber <gh@maxhbr.de>
Parts:
- removed the D1 at (161.9, 117.0)
- removed the D11 at (47.6, 72.6)
- removed the D12 at (85.7, 108.1)
- removed the D13 at (85.7, 96.2)
- removed the D14 at (85.7, 77.4)
- removed the D15 at (75.6, 61.9)
- removed the D2 at (161.9, 106.6)
- removed D20: BAV70, Package_TO_SOT_SMD:SOT-23
- removed the D3 at (161.9, 88.1)
- removed the D4 at (161.9, 69.1)
- removed the D5 at (103.0, 62.5)
- removed the D6 at (63.1, 114.9)
- removed the D7 at (123.8, 119.4)
- removed the D8 at (123.8, 102.4)
- removed the D9 at (123.8, 83.3)
- removed the FID2 at (32.1, 275.1)
- removed FID3 (x2): Fiducial, Fiducial:Fiducial_1mm_Mask2mm
- added L_D1: BAV70, Package_TO_SOT_SMD:SOT-23, B.Cu at (161.9, 118.5)
- added L_D10: BAV70, Package_TO_SOT_SMD:SOT-23, B.Cu at (79.8, 72.0)
- added L_D11: BAV70, Package_TO_SOT_SMD:SOT-23, B.Cu at (47.0, 72.0)
- added L_D12: BAV70, Package_TO_SOT_SMD:SOT-23, B.Cu at (85.7, 108.3)
- added L_D13: BAV70, Package_TO_SOT_SMD:SOT-23, B.Cu at (85.7, 91.1)
- added L_D14: BAV70, Package_TO_SOT_SMD:SOT-23, B.Cu at (85.7, 72.0)
- added L_D15: BAV70, Package_TO_SOT_SMD:SOT-23, B.Cu at (73.8, 72.0)
- added L_D2: BAV70, Package_TO_SOT_SMD:SOT-23, B.Cu at (161.9, 100.3)
- added L_D3: BAV70, Package_TO_SOT_SMD:SOT-23, B.Cu at (161.9, 80.7)
- added L_D4: BAV70, Package_TO_SOT_SMD:SOT-23, B.Cu at (161.9, 61.7)
- added L_D5: BAV70, Package_TO_SOT_SMD:SOT-23, B.Cu at (91.7, 71.8)
- added L_D6: BAV70, Package_TO_SOT_SMD:SOT-23, B.Cu at (63.1, 114.9)
- added L_D7: BAV70, Package_TO_SOT_SMD:SOT-23, B.Cu at (123.8, 114.3)
- added L_D8: BAV70, Package_TO_SOT_SMD:SOT-23, B.Cu at (123.8, 102.4)
- added L_D9: BAV70, Package_TO_SOT_SMD:SOT-23, B.Cu at (123.8, 97.0)
- added L_S1: SW_Push, pretty:PushSW, F.Cu at (167.0, 139.3)
- FID1: moved to F.Cu
- moved FID2 137.7 mm to (58.3, 151.2), turned to -90 degrees
- moved FID1 120.7 mm to (58.3, 139.9), turned to 90 degrees
- moved D15 52.3 mm to (73.8, 219.1), turned to 90 degrees
- moved FID1 23.7 mm to (161.3, 145.9)
- moved D5 14.6 mm to (91.7, 219.3)
- moved D10 10.9 mm to (79.8, 219.1), turned to 90 degrees
- moved D3 7.40 mm to (161.9, 210.4), turned to 90 degrees
- moved D4 7.40 mm to (161.9, 229.4), turned to 90 degrees
- moved D9 6.55 mm to (123.8, 201.2), turned to 90 degrees
- moved D2 6.30 mm to (161.9, 190.8), turned to 90 degrees
- moved D14 5.36 mm to (85.7, 219.1), turned to 90 degrees
- moved D13 5.10 mm to (85.7, 200.0), turned to 90 degrees
- moved D8 4.17 mm to (123.8, 192.9), turned to 90 degrees
- moved D1 1.44 mm to (161.9, 172.6), turned to 90 degrees
- moved D11 0.84 mm to (47.0, 219.1), turned to 90 degrees
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- renumbered D15 to D10, D20 to D15
Connections:
- D10 pad 1: Net-(D15-A1) -> Net-(D10-A1)
- D10 pad 2: Net-(D15-A2) -> Net-(D10-A2)
- D15 pad 1: Net-(D20-A1) -> Net-(D15-A1)
- D15 pad 2: Net-(D20-A2) -> Net-(D15-A2)
- L_S0 pad 1: COL0 -> L_COL0
- L_S0 pad 2: Net-(D1-A1) -> Net-(L_D1-A1)
- L_S10 pad 1: COL0 -> L_COL0
- L_S10 pad 2: Net-(D2-A1) -> Net-(L_D2-A1)
- L_S11 pad 1: COL1 -> L_COL1
- L_S11 pad 2: Net-(D2-A2) -> Net-(L_D2-A2)
- L_S12 pad 1: Net-(D7-A1) -> Net-(L_D7-A1)
- L_S12 pad 2: COL2 -> L_COL2
- L_S13 pad 1: COL3 -> L_COL3
- L_S13 pad 2: Net-(D7-A2) -> Net-(L_D7-A2)
- L_S14 pad 1: Net-(D12-A1) -> Net-(L_D12-A1)
- L_S14 pad 2: COL4 -> L_COL4
- L_S15 pad 1: COL5 -> L_COL5
- L_S15 pad 2: Net-(D12-A2) -> Net-(L_D12-A2)
- L_S2 pad 1: Net-(D6-A1) -> Net-(L_D6-A1)
- L_S2 pad 2: COL2 -> L_COL2
- L_S20 pad 1: COL0 -> L_COL0
- L_S20 pad 2: Net-(D3-A1) -> Net-(L_D3-A1)
- L_S21 pad 1: Net-(D3-A2) -> Net-(L_D3-A2)
- L_S21 pad 2: COL1 -> L_COL1
- L_S22 pad 1: COL2 -> L_COL2
- L_S22 pad 2: Net-(D8-A1) -> Net-(L_D8-A1)
- L_S23 pad 1: Net-(D8-A2) -> Net-(L_D8-A2)
- L_S23 pad 2: COL3 -> L_COL3
- L_S24 pad 1: COL4 -> L_COL4
- L_S24 pad 2: Net-(D13-A1) -> Net-(L_D13-A1)
- L_S25 pad 1: Net-(D13-A2) -> Net-(L_D13-A2)
- L_S25 pad 2: COL5 -> L_COL5
- L_S3 pad 1: COL3 -> L_COL3
- L_S3 pad 2: Net-(D6-A2) -> Net-(L_D6-A2)
- L_S30 pad 1: COL0 -> L_COL0
- L_S30 pad 2: Net-(D4-A1) -> Net-(L_D4-A1)
- L_S31 pad 1: Net-(D4-A2) -> Net-(L_D4-A2)
- L_S31 pad 2: COL1 -> L_COL1
- L_S32 pad 1: COL2 -> L_COL2
- L_S32 pad 2: Net-(D9-A1) -> Net-(L_D9-A1)
- L_S33 pad 1: Net-(D9-A2) -> Net-(L_D9-A2)
- L_S33 pad 2: COL3 -> L_COL3
- L_S34 pad 1: COL4 -> L_COL4
- L_S34 pad 2: Net-(D14-A1) -> Net-(L_D14-A1)
- L_S35 pad 1: Net-(D14-A2) -> Net-(L_D14-A2)
- L_S35 pad 2: COL5 -> L_COL5
- L_S4 pad 1: COL4 -> L_COL4
- L_S4 pad 2: Net-(D11-A1) -> Net-(L_D11-A1)
- L_S40 pad 1: COL0 -> L_COL0
- L_S40 pad 2: Net-(D5-A1) -> Net-(L_D5-A1)
- L_S42 pad 1: COL2 -> L_COL2
- L_S42 pad 2: Net-(D15-A1) -> Net-(L_D10-A1)
- L_S43 pad 1: Net-(D15-A2) -> Net-(L_D10-A2)
- L_S43 pad 2: COL3 -> L_COL3
- L_S44 pad 1: COL4 -> L_COL4
- L_S44 pad 2: Net-(D20-A1) -> Net-(L_D15-A1)
- L_S5 pad 1: Net-(D11-A2) -> Net-(L_D11-A2)
- L_S5 pad 2: COL5 -> L_COL5
- L_U1 pad 1: L_ROW1 -> L_ROW0
- L_U1 pad 2: L_ROW2 -> L_ROW1
- L_U1 pad 3: L_ROW3 -> L_ROW2
- L_U1 pad 4: L_ROW4 -> L_ROW3
- L_U1 pad 5: L_ROW5 -> L_ROW4
- S0 pad 1: COL0 -> Net-(D1-A1)
- S0 pad 2: Net-(D1-A1) -> COL0
- S1 pad 1: Net-(D1-A2) -> COL1
- S1 pad 2: COL1 -> Net-(D1-A2)
- S10 pad 1: COL0 -> Net-(D2-A1)
- S10 pad 2: Net-(D2-A1) -> COL0
- S11 pad 1: COL1 -> Net-(D2-A2)
- S11 pad 2: Net-(D2-A2) -> COL1
- S12 pad 1: Net-(D7-A1) -> COL2
- S12 pad 2: COL2 -> Net-(D7-A1)
- S13 pad 1: COL3 -> Net-(D7-A2)
- S13 pad 2: Net-(D7-A2) -> COL3
- S14 pad 1: Net-(D12-A1) -> COL4
- S14 pad 2: COL4 -> Net-(D12-A1)
- S15 pad 1: COL5 -> Net-(D12-A2)
- S15 pad 2: Net-(D12-A2) -> COL5
- S2 pad 1: Net-(D6-A1) -> COL2
- S2 pad 2: COL2 -> Net-(D6-A1)
- S20 pad 1: COL0 -> Net-(D3-A1)
- S20 pad 2: Net-(D3-A1) -> COL0
- S21 pad 1: Net-(D3-A2) -> COL1
- S21 pad 2: COL1 -> Net-(D3-A2)
- S22 pad 1: COL2 -> Net-(D8-A1)
- S22 pad 2: Net-(D8-A1) -> COL2
- S23 pad 1: Net-(D8-A2) -> COL3
- S23 pad 2: COL3 -> Net-(D8-A2)
- S24 pad 1: COL4 -> Net-(D13-A1)
- S24 pad 2: Net-(D13-A1) -> COL4
- S25 pad 1: Net-(D13-A2) -> COL5
- S25 pad 2: COL5 -> Net-(D13-A2)
- S3 pad 1: COL3 -> Net-(D6-A2)
- S3 pad 2: Net-(D6-A2) -> COL3
- S30 pad 1: COL0 -> Net-(D4-A1)
- S30 pad 2: Net-(D4-A1) -> COL0
- S31 pad 1: Net-(D4-A2) -> COL1
- S31 pad 2: COL1 -> Net-(D4-A2)
- S32 pad 1: COL2 -> Net-(D9-A1)
- S32 pad 2: Net-(D9-A1) -> COL2
- S33 pad 1: Net-(D9-A2) -> COL3
- S33 pad 2: COL3 -> Net-(D9-A2)
- S34 pad 1: COL4 -> Net-(D14-A1)
- S34 pad 2: Net-(D14-A1) -> COL4
- S35 pad 1: Net-(D14-A2) -> COL5
- S35 pad 2: COL5 -> Net-(D14-A2)
- S4 pad 1: COL4 -> Net-(D11-A1)
- S4 pad 2: Net-(D11-A1) -> COL4
- S40 pad 1: COL0 -> Net-(D5-A1)
- S40 pad 2: Net-(D5-A1) -> COL0
- S42 pad 1: COL2 -> Net-(D10-A1)
- S42 pad 2: Net-(D15-A1) -> COL2
- S43 pad 1: Net-(D15-A2) -> COL3
- S43 pad 2: COL3 -> Net-(D10-A2)
- S44 pad 1: COL4 -> Net-(D15-A1)
- S44 pad 2: Net-(D20-A1) -> COL4
- S5 pad 1: Net-(D11-A2) -> COL5
- S5 pad 2: COL5 -> Net-(D11-A2)
- U1 pad 1: ROW1 -> ROW0
- U1 pad 2: ROW2 -> ROW1
- U1 pad 3: ROW3 -> ROW2
- U1 pad 4: ROW4 -> ROW3
- U1 pad 5: ROW5 -> ROW4
- locked pad 1: Net-(D20-A2) -> COL5
- locked pad 2: COL5 -> Net-(D15-A2)
- locked pad 1: Net-(D5-A2) -> Net-(L_D5-A2)
- locked pad 2: COL1 -> L_COL1
- locked pad 1: Net-(D20-A2) -> Net-(L_D15-A2)
- locked pad 2: COL5 -> L_COL5
- locked pad 1: Net-(D5-A2) -> COL1
- locked pad 2: COL1 -> Net-(D5-A2)
Routing:
- net COL3: track 13.3 -> 272.0 mm
- net COL5: track 9.73 -> 265.3 mm
- net L_COL5: track 9.73 -> 234.3 mm
- net COL4: track 11.7 -> 228.9 mm
- net L_COL1: track 10.2 -> 217.3 mm, vias 0 -> 2
- net L_COL3: track 13.3 -> 214.5 mm, vias 2 -> 5
- net L_ROW0: track 0.00 -> 194.5 mm, vias 0 -> 2
- net ROW0: track 0.00 -> 192.4 mm, vias 0 -> 3
- net COL2: track 12.1 -> 202.8 mm
- net L_COL4: track 11.7 -> 197.4 mm, vias 2 -> 7
- net ROW3: track 14.7 -> 198.0 mm, vias 0 -> 1
- net ROW4: track 11.5 -> 177.5 mm, vias 0 -> 1
- net COL1: track 10.2 -> 151.9 mm, vias 0 -> 1
- net L_ROW4: track 11.5 -> 153.1 mm, vias 0 -> 3
- net ROW2: track 16.4 -> 156.8 mm, vias 0 -> 1
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