File: mykeeb/rev7/mykeeb_v7a3/mykeeb_v7a3.kicad_sch (KiCad schematic)
At the start: 62 parts, among them SW44 SW_SPDT, U1 74HC595, U2 xiao-ble

Commit message: finalize v7a3 for now
Signed-off-by: Maximilian Huber <gh@maxhbr.de>
Other:
- moved on the sheet: BT1, D1, D11, D12, D13, D14, D15, D2, D3, D4, D6, D7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
