File: mykeeb/rev7/mykeeb_v7a3/mykeeb_v7a3.kicad_pcb (KiCad board)
At the start: 2 copper layers, 160.4 x 147.9 mm, 62 parts, among them U1 xiao-ble, U2 74HC595, U3 74HC595

Commit message: finalize v7a3 for now
Signed-off-by: Maximilian Huber <gh@maxhbr.de>
Connections:
- U1 pad 6: rowF -> unconnected-(U1-A9_SCL/0.05_H-Pad6)
- U1 pad 7: rowG -> unconnected-(U1-B8_TX/1.11-Pad7)
Routing:
- net unconnected-(U1-A9_SCL/0.05_H-Pad6): track 0.00 -> 35.8 mm, vias 0 -> 1
- net rowF: track 35.8 -> 0.00 mm, vias 1 -> 0
- net unconnected-(U1-B8_TX/1.11-Pad7): track 0.00 -> 28.4 mm, vias 0 -> 1
- net rowG: track 28.4 -> 0.00 mm, vias 1 -> 0
- net Net-(D16-A1): track 50.1 -> 47.5 mm
- net GND: track 27.5 -> 28.0 mm, vias 85 -> 84
Other:
- board text added: "locked"
- board text removed: "github.com/maxhbr"

Commit message: add plates
Signed-off-by: Maximilian Huber <gh@maxhbr.de>
Routing:
- net rowA: track 169.8 -> 192.9 mm

Commit message: update
Signed-off-by: Maximilian Huber <gh@maxhbr.de>
Routing:
- net Net-(D16-A1): track 47.5 -> 50.1 mm
- net Net-(D9-A1): track 30.9 -> 28.3 mm
- net Net-(D7-A1): track 30.3 -> 28.4 mm
- net rowA: track 192.9 -> 192.3 mm
- net GND: vias 84 -> 81
