File: mykeeb/rev7/mykeeb_v7a3/mykeeb_v7a3.kicad_pcb (KiCad board)
At the start: 2 copper layers, 160.4 x 147.9 mm, 62 parts, among them U1 xiao-ble, U2 74HC595, U3 74HC595

Commit message: update gerbers, step 1
Signed-off-by: Maximilian Huber <gh@maxhbr.de>
Parts:
- moved D19 0.24 mm to (108.3, 123.2)
Routing:
- net Net-(D12-A1): track 30.7 -> 28.7 mm
- net Net-(D11-A1): track 30.5 -> 28.7 mm
- net Net-(D1-A2): track 17.8 -> 19.4 mm
- net Net-(D13-A1): track 31.0 -> 31.5 mm
- net GND: vias 81 -> 79

Commit message: update
Signed-off-by: Maximilian Huber <gh@maxhbr.de>
Parts:
- moved D10 3.57 mm to (123.2, 120.3)
Routing:
- net Net-(D10-A1): track 28.3 -> 31.8 mm
- net Net-(D10-A2): track 42.5 -> 38.9 mm
- net Net-(D1-A2): track 19.4 -> 18.1 mm
- net GND: vias 79 -> 81
