File: mykeeb/rev7/mykeeb_v7a5/mykeeb_v7a5.kicad_pcb (KiCad board)
At the start: 2 copper layers, 162.3 x 124.3 mm, 64 parts, among them Q1 AO3416 N-channel MOSFET, SW1 SW_Push, U1 xiao-ble, U2 74HC595

Commit message: work on v7a5
Signed-off-by: Maximilian Huber <gh@maxhbr.de>
Parts:
- removed JP1: SolderJumper_3_Open, Jumper:SolderJumper-3_P1.3mm_Open_RoundedPad1.0x1.5mm
- removed LED1, LED2: YS-SK6812MINI-E, pretty:LED_SK6812-MINI-E
- removed LED3, LED4, LED5, LED6, LED7, LED8: WS2812B, LED_SMD:LED_WS2812B_PLCC4_5.0x5.0mm_P3.2mm
- removed Q1: AO3416 N-channel MOSFET, Package_TO_SOT_SMD:SOT-23
- removed R1: 4.7k, Resistor_SMD:R_1206_3216Metric_Pad1.30x1.75mm_HandSolder
- removed R_A1, R_A2: R, Resistor_SMD:R_1206_3216Metric_Pad1.30x1.75mm_HandSolder
- removed U2: 74HC595, Package_SO:SOIC-16_3.9x9.9mm_P1.27mm
- added D4: BAV70, Package_TO_SOT_SMD:SOT-23, B.Cu at (42.3, 57.7)
- added R_BT1: Battery_Cell, Connector_JST:JST_PH_S2B-PH-K_1x02_P2.00mm_Horizontal, B.Cu at (286.3, 114.3)
- added R_D1: BAV70, pretty:SOT-23, B.Cu at (320.9, 73.8)
- added R_D10: BAV70, pretty:SOT-23, B.Cu at (231.6, 128.0)
- added R_D11: BAV70, pretty:SOT-23, B.Cu at (244.7, 65.5)
- added R_D12: BAV70, pretty:SOT-23, B.Cu at (244.7, 84.5)
- added R_D13: BAV70, pretty:SOT-23, B.Cu at (244.7, 103.6)
- added R_D14: BAV70, pretty:SOT-23, B.Cu at (221.5, 97.3)
- added R_D15: BAV70, pretty:SOT-23, B.Cu at (214.9, 140.5)
- added R_D2: BAV70, pretty:SOT-23, B.Cu at (320.9, 92.9)
- added R_D3: BAV70, pretty:SOT-23, B.Cu at (320.9, 111.9)
- added R_D4: BAV70, Package_TO_SOT_SMD:SOT-23, B.Cu at (326.8, 57.7)
- added R_D5: BAV70, pretty:SOT-23, B.Cu at (279.2, 128.6)
- added R_D6: BAV70, pretty:SOT-23, B.Cu at (282.8, 56.0)
- added R_D7: BAV70, pretty:SOT-23, B.Cu at (282.8, 75.0)
- added R_D8: BAV70, pretty:SOT-23, B.Cu at (282.8, 94.1)
- added R_D9: BAV70, pretty:SOT-23, B.Cu at (221.5, 81.6)
- added R_SA0: SW, pretty:CherryMX_Hotswap, F.Cu at (341.0, 70.8)
- added R_SA1: SW, pretty:CherryMX_Hotswap, F.Cu at (320.9, 69.7)
- added R_SA2: SW, pretty:CherryMX_Hotswap, F.Cu at (301.8, 57.7)
- added R_SA3: SW, pretty:CherryMX_Hotswap, F.Cu at (282.8, 51.8)
- added R_SA4: SW, pretty:CherryMX_Hotswap, F.Cu at (263.7, 58.9)
- added R_SA5: SW, pretty:CherryMX_Hotswap, F.Cu at (244.7, 61.3)
- added R_SB0: SW, pretty:CherryMX_Hotswap, F.Cu at (341.0, 90.0)
- added R_SB1: SW, pretty:CherryMX_Hotswap, F.Cu at (320.9, 88.7)
- added R_SB2: SW, pretty:CherryMX_Hotswap, F.Cu at (301.8, 76.8)
- added R_SB3: SW, pretty:CherryMX_Hotswap, F.Cu at (282.8, 70.8)
- added R_SB4: SW, pretty:CherryMX_Hotswap, F.Cu at (263.7, 78.0)
- added R_SB5: SW, pretty:CherryMX_Hotswap, F.Cu at (244.7, 80.4)
- added R_SC0: SW, pretty:CherryMX_Hotswap, F.Cu at (339.9, 110.1)
- added R_SC1: SW, pretty:CherryMX_Hotswap, F.Cu at (320.9, 107.8)
- added R_SC2: SW, pretty:CherryMX_Hotswap, F.Cu at (301.8, 95.8)
- added R_SC3: SW, pretty:CherryMX_Hotswap, F.Cu at (282.8, 89.9)
- added R_SC4: SW, pretty:CherryMX_Hotswap, F.Cu at (263.7, 97.0)
- added R_SC5: SW, pretty:CherryMX_Hotswap, F.Cu at (244.7, 99.4)
- added R_SD0: SW_Push, pretty:PushSW, F.Cu at (339.3, 48.2)
- added R_SD1: SW_Push, pretty:PushSW, F.Cu at (313.7, 53.9)
- added R_SD2: SW, pretty:CherryMX_Hotswap, F.Cu at (225.6, 60.1)
- added R_SD3: SW, pretty:CherryMX_1.25U_Hotswap, F.Cu at (225.6, 81.6)
- added R_SD4: SW, pretty:CherryMX_1.25U_Hotswap, F.Cu at (219.7, 107.9)
- added R_SD5: SW, pretty:CherryMX_1.25U_Hotswap, F.Cu at (198.5, 124.0)
- added R_SE0: SW, pretty:CherryMX_Hotswap, F.Cu at (301.8, 114.9)
- added R_SE0_alt1: SW_Push, Button_Switch_THT:SW_Tactile_SPST_Angled_PTS645Vx39-2LFS, F.Cu at (304.1, 119.8)
- added R_SE2: SW, pretty:CherryMX_1.25U_Hotswap, F.Cu at (254.2, 118.5)
- added R_SE3: SW, pretty:CherryMX_Hotswap, F.Cu at (229.2, 124.4)
- added R_SE4: SW, pretty:CherryMX_Hotswap, F.Cu at (211.9, 137.5)
- added R_SW1: SW_Push, Button_Switch_SMD:SW_SPST_TL3342, B.Cu at (326.8, 51.2)
- added R_SW_bat1: SW_SPDT, sepp:switch-MSK-12C02-smd, B.Cu at (254.2, 125.0)
- added R_U1: xiao-ble, pretty:xiao-ble-smd-cutout, B.Cu at (326.8, 51.8)
- added SD0: SW_Push, pretty:PushSW, F.Cu at (29.8, 48.2)
- added SD1: SW_Push, pretty:PushSW, F.Cu at (55.4, 53.9)
- added locked: SW, pretty:CherryMX_Hotswap, F.Cu at (279.2, 124.4)
- added locked: SW, pretty:CherryMX_Hotswap, F.Cu at (198.8, 154.8)
- BT1, SE0_alt1: moved to F.Cu
- moved SE0_alt1 4.55 mm to (69.5, 119.8), turned to 180 degrees
- moved BT1 1.60 mm to (82.8, 114.3), turned to -90 degrees
- moved SW_bat1 0.20 mm to (114.9, 125.0)
Connections:
- SE0_alt1 pad 1: col0 -> Net-(D5-A1)
- SE0_alt1 pad 2: Net-(D5-A1) -> col0
- U1 pad 10: MISO -> col1
- U1 pad 11: MOSI -> col0
- U1 pad 12: +3V3 -> unconnected-(U1-3V3-Pad12)
- U1 pad 14: Net-(JP1-B) -> unconnected-(U1-5V-Pad14)
- U1 pad 5: unconnected-(U1-A8_SDA/0.04_H-Pad5) -> rowE
- U1 pad 6: unconnected-(U1-A9_SCL/0.05_H-Pad6) -> col5
- U1 pad 7: rowE -> col4
- U1 pad 8: ledTrig -> col3
- U1 pad 9: SCK -> col2
Routing:
- net R_rowC: track 0.00 -> 98.1 mm
- net R_rowA: track 0.00 -> 97.7 mm
- net R_rowB: track 0.00 -> 97.1 mm
- net +3V3: track 94.1 -> 0.00 mm, vias 1 -> 0
- net MOSI: track 83.9 -> 0.00 mm, vias 1 -> 0
- net MISO: track 79.6 -> 0.00 mm, vias 1 -> 0
- net SCK: track 77.8 -> 0.00 mm, vias 1 -> 0
- net rowC: track 160.1 -> 232.0 mm, vias 1 -> 2
- net rowB: track 136.5 -> 204.5 mm, vias 1 -> 2
- net col1: track 132.1 -> 197.5 mm, vias 0 -> 2
- net R_col0: track 0.00 -> 42.8 mm
- net rowE: track 179.4 -> 221.4 mm, vias 1 -> 0
- net Net-(D4-A2): track 0.00 -> 40.8 mm
- net Net-(R_D5-A1): track 0.00 -> 38.4 mm
- net Net-(R_D11-A1): track 0.00 -> 33.9 mm
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- added copper zone on B.Cu, net R_GND
- added copper zone on F.Cu, net R_GND
Other:
- board size 162.3 x 124.3 mm -> 329.8 x 124.3 mm

Commit message: openscad? -> yes!
Signed-off-by: Maximilian Huber <gh@maxhbr.de>
Connections:
- R_SE0_alt1 pad 1: (no net) -> Net-(R_D5-A1)
- R_SE0_alt1 pad 2: (no net) -> R_col0
Routing:
- net R_col5: track 0.00 -> 267.6 mm, vias 0 -> 10
- net R_col2: track 0.00 -> 248.5 mm, vias 0 -> 6
- net R_col4: track 0.00 -> 248.2 mm, vias 0 -> 8
- net R_col3: track 0.00 -> 218.8 mm, vias 0 -> 4
- net R_rowE: track 25.0 -> 227.4 mm
- net R_rowD: track 12.8 -> 158.7 mm, vias 0 -> 3
- net R_col1: track 0.00 -> 137.4 mm, vias 0 -> 4
- net R_BAT+: track 0.00 -> 132.5 mm, vias 0 -> 2
- net R_col0: track 42.8 -> 172.0 mm, vias 0 -> 1
- net R_rowC: track 98.1 -> 198.1 mm, vias 0 -> 2
- net R_rowB: track 97.1 -> 167.6 mm, vias 0 -> 2
- net Net-(R_D4-A1): track 0.00 -> 43.0 mm
- net R_rowA: track 97.7 -> 136.1 mm
- net Net-(R_D10-A1): track 0.00 -> 37.5 mm
- net R_VBAT: track 0.00 -> 33.0 mm, vias 0 -> 1
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Other:
- board size 329.8 x 124.3 mm -> 337.5 x 131 mm
