File: mykeeb/rev7/mykeeb_v7a5/mykeeb_v7a5-base.kicad_pcb (KiCad board)
At the start: 2 copper layers, 175.6 x 131 mm, 0 parts

Commit message: add gerbers
Signed-off-by: Maximilian Huber <gh@maxhbr.de>
Other:
- board size 175.6 x 131 mm -> 165.5 x 125.7 mm
Changed lines of the file:
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@@
       (drillshape 0)
       (scaleselection 1)
-      (outputdirectory "gerber")
+      (outputdirectory "gerber-base")
     )
   )
@@
   (gr_arc locked (start 23.217207 119.657865) (mid 20.691497 118.611731) (end 19.645329 116.086035)
     (stroke (width 0.16) (type solid)) (layer "Edge.Cuts"))
-  (gr_rect (start 13.096886 164.306388) (end 17.264077 166.68764)
-    (stroke (width 0.0381) (type default)) (fill none) (layer "Edge.Cuts"))
   (gr_line locked (start 23.217207 119.657865) (end 25.598459 119.657913)
     (stroke (width 0.0381) (type default)) (layer "Edge.Cuts"))
   (gr_arc locked (start 17.85939 58.340674) (mid 18.905567 55.814973) (end 21.431268 54.768796)
     (stroke (width 0.1) (type default)) (layer "Edge.Cuts"))
-  (gr_rect (start 179.784526 38.100032) (end 186.332969 42.862536)
-    (stroke (width 0.0381) (type default)) (fill none) (layer "Edge.Cuts"))
   (gr_arc locked (start 26.789085 44.648475) (mid 27.835261 42.122773) (end 30.360963 41.076597)
     (stroke (width 0.1) (type default)) (layer "Edge.Cuts"))
@@
   (gr_line locked (start 105.965714 49.410979) (end 113.10947 49.410979)
     (stroke (width 0.1) (type default)) (layer "Edge.Cuts"))
-  (gr_rect (start 180.975152 39.290658) (end 185.142343 41.67191)
-    (stroke (width 0.0381) (type default)) (fill none) (layer "Edge.Cuts"))
-  (gr_rect (start 11.310947 162.520449) (end 19.050016 168.473579)
-    (stroke (width 0.0381) (type default)) (fill none) (layer "Edge.Cuts"))
   (gr_curve locked (pts (xy 116.132283 127.928273) (xy 104.226023 127.928273) (xy 101.249458 129.714212) (xy 89.29695 136.326677))
     (stroke (width 0.16) (type solid)) (layer "Edge.Cuts"))
@@
   (gr_circle locked (center 25.598459 58.340674) (end 26.789085 58.340674)
     (stroke (width 0.0381) (type default)) (fill none) (layer "Edge.Cuts"))
-  (gr_rect (start 11.90626 163.115762) (end 18.454703 167.878266)
-    (stroke (width 0.0381) (type default)) (fill none) (layer "Edge.Cuts"))
   (gr_circle locked (center 175.617335 138.707929) (end 176.807961 138.707929)
-    (stroke (width 0.0381) (type default)) (fill none) (layer "Edge.Cuts"))
-  (gr_rect (start 13.692199 164.901701) (end 16.668764 166.092327)
     (stroke (width 0.0381) (type default)) (fill none) (layer "Edge.Cuts"))
   (gr_arc locked (start 89.29695 136.326677) (mid 86.586607 136.683644) (end 84.417666 135.019586)
@@
   (gr_line locked (start 147.042311 50.601605) (end 149.423563 50.601605)
     (stroke (width 0.0381) (type default)) (layer "Edge.Cuts"))
-  (gr_rect (start 179.189213 37.504719) (end 186.928282 43.457849)
-    (stroke (width 0.0381) (type default)) (fill none) (layer "Edge.Cuts"))
   (gr_arc locked (start 182.251803 122.27575) (mid 183.069862 123.538602) (end 183.356404 125.01573)
     (stroke (width 0.16) (type solid)) (layer "Edge.Cuts"))
-  (gr_rect (start 181.570465 39.885971) (end 184.54703 41.076597)
-    (stroke (width 0.0381) (type default)) (fill none) (layer "Edge.Cuts"))
   (gr_line locked (start 182.445562 156.9004) (end 183.356404 125.01573)
     (stroke (width 0.0381) (type default)) (layer "Edge.Cuts"))
