File: mykeeb/rev7/mykeeb_v7a5/mykeeb_v7a5.kicad_sch (KiCad schematic)
At the start: 66 parts, among them Q1 AO3416 N-channel MOSFET, SW43 SW_Push, SW44 SW_SPDT, U1 74HC595, U2 xiao-ble

Commit message: work on v7a5
Signed-off-by: Maximilian Huber <gh@maxhbr.de>
Parts:
- removed D20, D21: LED, symbol Device:LED
- removed JP1: SolderJumper_3_Open, Jumper:SolderJumper-3_P1.3mm_Open_RoundedPad1.0x1.5mm, symbol 41_1350_pcb-rescue:SolderJumper_3_Open-Jumper
- removed LED1, LED2: YS-SK6812MINI-E, pretty:LED_SK6812-MINI-E, symbol zzkeeb:LED_SK6812MINI-E
- removed LED1, LED2, LED3, LED4, LED5, LED6: WS2812B, LED_SMD:LED_WS2812B_PLCC4_5.0x5.0mm_P3.2mm, symbol LED:WS2812B
- removed Q1: AO3416 N-channel MOSFET, Package_TO_SOT_SMD:SOT-23, symbol Device:Q_NMOS_GSD
- removed R80: 4.7k, Resistor_SMD:R_1206_3216Metric_Pad1.30x1.75mm_HandSolder, symbol Device:R_US
- removed R_A0 (x2): R, Resistor_SMD:R_1206_3216Metric_Pad1.30x1.75mm_HandSolder, symbol Device:R_Small_US
- removed U1: 74HC595, Package_SO:SOIC-16_3.9x9.9mm_P1.27mm, symbol 74xx:74HC595
- added BT1: Battery_Cell, Connector_JST:JST_PH_S2B-PH-K_1x02_P2.00mm_Horizontal, symbol Device:Battery_Cell
- added D1 (x2): BAV70, Package_TO_SOT_SMD:SOT-23, symbol hillside_basic:BAV70_Small
- added D1, D11, D12, D13, D15 (x2), D2, D3, D4 (x2), D6, D7, D8, D9: BAV70, pretty:SOT-23, symbol hillside_basic:BAV70_Small
- added S0, S1, S10, S11, S12, S13, S14, S15, S2 (x2), S20, S21, S22, S23, S24, S25, S3, S30, S4, S43, S45 (x3), S46: SW, pretty:CherryMX_Hotswap, symbol YAEMK:MX_1U
- added S31, S32, S33, S44: SW, pretty:CherryMX_1.25U_Hotswap, symbol YAEMK:MX_1U
- added SW43: SW_Push, Button_Switch_THT:SW_Tactile_SPST_Angled_PTS645Vx39-2LFS, symbol Switch:SW_Push
- added SW43 (x4): SW_Push, pretty:PushSW, symbol Switch:SW_Push
- added SW43: SW_Push, Button_Switch_SMD:SW_SPST_TL3342, symbol Switch:SW_Push
- added SW44: SW_SPDT, sepp:switch-MSK-12C02-smd, symbol Switch:SW_SPDT
- added U2: xiao-ble, pretty:xiao-ble-smd-cutout, symbol sepp:xiao-ble-geist
Connections:
- net MISO is gone; now on net col1: U2.10 (A5_MISO/1.14)
- net MOSI is gone; now on net col0: U2.11 (A6_MOSI/1.15)
- net SCK is gone; now on net col2: U2.9 (A7_SCK/1.13)
- net ledTrig is gone; now on net col3: U2.8 (B9_RX/1.12)
- net col0: now also SW43.2, SW43.1; no longer SW43.1
- net col1: now also SW43.2
- net col4: now also U2.7 (B8_TX/1.11)
- net col5: now also U2.6 (A9_SCL/0.05_H)
- net rowD: now also D1.3 (K)
- net rowE: now also U2.5 (A8_SDA/0.04_H); no longer U2.7 (B8_TX/1.11)
- net at D4.1 (A1), S45.2: now also SW43.1; no longer SW43.2
- net +3V3: no longer names the net of U2.12 (3V3)
- new net: D6.2 (A2), S3.1
- new net: D2.2 (A2), S11.1
- new net: D1.1 (A1), SW43.2 (x2)
- new net: D1.2 (A2), SW43.1 (x2)
- new net: D15.2 (A2), S45.1 (x2)
- new net: D1.1 (A1), S0.2
- new net: D6.1 (A1), S2.2
- new net: D13.2 (A2), S25.1
- new net: D12.1 (A1), S14.2
- new net: D12.2 (A2), S15.1
- new net: D3.1 (A1), S20.2
- new net: D15.1 (A1), S44.2
- new net: D3.2 (A2), S21.1
- new net: D15.1 (A1), S46.2
- new net: D4.1 (A1), S30.2
- new net: D4.2 (A2), S31.1
- new net: D4.1 (A1), S45.2, SW43.1
- new net: D4.2 (A2), S43.1
- new net: D2.1 (A1), S10.2
- new net: D13.1 (A1), S24.2
- new net: D8.2 (A2), S23.1
- new net: D7.1 (A1), S12.2
- new net: D7.2 (A2), S13.1
- new net: D11.1 (A1), S4.2
- new net: D9.1 (A1), S32.2
- new net: D11.2 (A2), S1.1
- new net: D9.2 (A2), S33.1
- new net: D1.2 (A2), S2.1
- new net: D8.1 (A1), S22.2
- new net R_BAT+: SW44.2 (B), U2.19 (BAT)
- new net R_GND: SW43.2, U2.13 (GND), U2.18 (GND), U2.20 (GND)
- new net R_RESET: SW43.1, U2.17 (RESET)
- new net R_VBAT: BT1.1 (+), SW44.1 (A)
- new net R_col0: S0.1, S10.1, S20.1, S45.1, SW43.1, SW43.2, U2.11 (A6_MOSI/1.15)
- new net R_col1: S11.2, S2.2, S21.2, S43.2, SW43.2, U2.10 (A5_MISO/1.14)
- new net R_col2: S12.1, S2.1, S22.1, S30.1, S44.1, U2.9 (A7_SCK/1.13)
- new net R_col3: S13.2, S23.2, S3.2, S31.2, S45.2, U2.8 (B9_RX/1.12)
- new net R_col4: S14.1, S24.1, S32.1, S4.1, S46.1, U2.7 (B8_TX/1.11)
- new net R_col5: S1.2, S15.2, S25.2, S33.2, S45.2, U2.6 (A9_SCL/0.05_H)
- new net R_rowA: D1.3 (K), D11.3 (K), D6.3 (K), U2.1 (A2/0.02_H)
- new net R_rowB: D12.3 (K), D2.3 (K), D7.3 (K), U2.2 (A4/0.03_H)
- new net R_rowC: D13.3 (K), D3.3 (K), D8.3 (K), U2.3 (A10/0.28)
- new net R_rowD: D1.3 (K), D4.3 (K), D9.3 (K), U2.4 (A11/0.29)
- new net R_rowE: D15.3 (K), D15.3 (K), D4.3 (K), U2.5 (A8_SDA/0.04_H)
- no-connect marks 7 -> 10
Other:
- moved on the sheet: BT1, SW43, SW44, U2

Commit message: fix the small 'MCU on the wrong side' issue
Signed-off-by: Maximilian Huber <gh@maxhbr.de>
Parts:
- removed D1 (x2): BAV70, Package_TO_SOT_SMD:SOT-23, symbol hillside_basic:BAV70_Small
- removed SW43 (x4): SW_Push, pretty:PushSW, symbol Switch:SW_Push
- added MB1, MB2, MB3, MB4, MB5, MB6: Mousebites, pretty:mousebites, symbol Mechanical:Heatsink

Commit message: update pcb after messup
Signed-off-by: Maximilian Huber <gh@maxhbr.de>
Connections:
- net R_GND: now also BT1.2 (-)
Changed lines of the file:
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@@
     )
   )
-  (global_label "R_GND" (shape input) (at 236.855 99.695 270) (fields_autoplaced)
+  (global_label "R_GND" (shape input) (at 236.855 99.06 270) (fields_autoplaced)
     (effects (font (size 1.27 1.27)) (justify right))
-    (property "Intersheetrefs" "${INTERSHEET_REFS}" (at 236.855 108.7089 90)
+    (property "Intersheetrefs" "${INTERSHEET_REFS}" (at 236.855 108.0739 90)
       (effects (font (size 1.27 1.27)) (justify right) hide)
     )
